File: hardware/dock/usb_keyboard_host.kicad_sch (KiCad schematic)
At the start: 0 parts

Commit message: Dock schematic: review fixes, Pico 2/XIAO socket+pogo mounting
- Cross HID UART TX/RX; split ROLE_STRAP per endpoint
- VBUS sense (GP4) and USB-C CC current sensing (GP26/27) on HID endpoints
- Pogo +5V via TPS2552 enabled by DET, TPD4E1U06 ESD + 1k on pogo lines
- 2x100uF bulk on SYS_5V and keyboard VBUS; 100k EN pull-down
- Remove TPS62162 rail: XIAO from 5V, pull-ups on module 3V3 rails
- Socketed Pico 2 / XIAO footprints with P50-B1 probe holes for USB+SWD
- XIAO SWD header J8; RP2350 reset control of HID/BLE endpoints
- DESIGN.md: UART allocation, power budget, mounting, reset control
- Add .gitignore, custom libraries and datasheets

Co-Authored-By: Claude Opus 5.5 <noreply@anthropic.com>
Parts:
- added C1: 100nF, Capacitor_SMD:C_0805_2012Metric_Pad1.18x1.45mm_HandSolder, symbol Device:C
- added C15, C16: 100uF, Capacitor_SMD:CP_Elec_6.3x7.7, symbol Device:C_Polarized
- added C6, C7: 1uF, Capacitor_SMD:C_0805_2012Metric_Pad1.18x1.45mm_HandSolder, symbol Device:C
- added J1: (no value), dock:KLS L-KLS1-5416-L1-01-R, symbol dock_custom:KLS_L-KLS1-5416-L1-01-R
- added R28: 100k, Resistor_SMD:R_0805_2012Metric_Pad1.20x1.40mm_HandSolder, symbol Device:R
- added R5: 26.1k, Resistor_SMD:R_0805_2012Metric_Pad1.20x1.40mm_HandSolder, symbol Device:R
- added R6: 10k, Resistor_SMD:R_0805_2012Metric_Pad1.20x1.40mm_HandSolder, symbol Device:R
- added R7, R8: 56k, Resistor_SMD:R_0805_2012Metric_Pad1.20x1.40mm_HandSolder, symbol Device:R
- added R9: 330, Resistor_SMD:R_0805_2012Metric_Pad1.20x1.40mm_HandSolder, symbol Device:R
- added U3: (no value), Package_TO_SOT_SMD:SOT-23-6, symbol dock_custom:TPS2553DBV
- added U4: TPD2EUSB30, Package_TO_SOT_SMD:Texas_DRT-3, symbol Power_Protection:TPD2EUSB30
Connections:
- new net: J1.4 (CC1_A5), R8.1
- new net: C1.2, J1.SH (SHIELD), R9.1
- new net: R5.1, U3.5 (ILIM)
- new net: J1.10 (CC2_B5), R7.1
- new net GND: C1.1, C15.2, C16.2, C6.1, C7.1, J1.1 (GND_A1_B12), J1.12 (GND_B1_A12), R28.2, R5.2, R9.2, U3.2 (GND), U4.3 (GND)
- new net HOST_3V3: R6.1
- new net KEYBOARD_VBUS: C15.1, C16.1, C7.2, J1.11 (VBUS_B4_A9), J1.2 (VBUS_A4_B9), R7.2, R8.2, U3.6 (OUT)
- new net KEYBOARD_VBUS_EN: R28.1, U3.3 (EN)
- new net KEYBOARD_VBUS_FAULT: R6.2, U3.4 (FAULT)
- new net SYS_5V: C6.2, U3.1 (IN)
- new net USB_HOST_DM: J1.5 (DM_B7), J1.7 (DM_A7), U4.2 (D-)
- new net USB_HOST_DP: J1.6 (DP_A6), J1.8 (DP_B6), U4.1 (D+)
- no-connect marks 0 -> 2

Commit message: Net classes, project lib tables, docs and datasheets; PCB synced
- Rename USB pairs to *_D_P/*_D_N; add Power and USB net classes
- Project-relative fp-lib-table and new sym-lib-table
- Pico values set to "Raspberry Pi Pico 2"; J1 symbol synced with library
- DESIGN.md/README: Pico 2 x3 + XIAO modules, TPS2116, pogo switch/ESD,
  VBUS/CC sensing, SWD pinout, resolved and open items
- Add TPS2552/2553, TPD2EUSB30 and P50 probe datasheets
- PCB updated from schematic (F8)

Co-Authored-By: Claude Opus 5.5 <noreply@anthropic.com>
Connections:
- net USB_HOST_DM renamed USB_HOST_D_N
- net USB_HOST_DP renamed USB_HOST_D_P

Commit message: USB ESD: TPD2EUSB30 -> TPD4E1U06 on all ports; Pico TP4-6 pads
- U4-U6 now TPD4E1U06 (SOT-23-6, hand-solderable): D+, D-, CC1, CC2
  per port; clamps to GND only, so no back-feed path into PC VBUS
- Keyboard port CC nets named CC1/CC2 (R7/R8 moved along their rows)
- Pico 2 footprint: TP4-TP6 as covered copper-only pads at datasheet
  positions (satisfies F8 pad check, no extra holes)
- Drop unused cached symbols; docs updated; remove TPD2EUSB30 datasheet

Co-Authored-By: Claude Opus 5.5 <noreply@anthropic.com>
Parts:
- U4: value TPD2EUSB30 -> TPD4E1U06DBVR; footprint Package_TO_SOT_SMD:Texas_DRT-3 -> Package_TO_SOT_SMD:SOT-23-6; symbol Power_Protection:TPD2EUSB30 -> dock_custom:TPD4E1U06DBV
Connections:
- net GND: now also U4.2 (GND); no longer U4.3 (GND)
- net USB_HOST_D_N: now also U4.6 (D1-); no longer U4.2 (D-)
- net CC1: now reaches J1.4 (CC1_A5), R8.1
- net CC1: now also U4.3 (D2+)
- net CC2: now reaches J1.10 (CC2_B5), R7.1
- net CC2: now also U4.4 (D2-)
- no-connect marks 2 -> 3
Other:
- moved on the sheet: R7, R8

Commit message: Set part values; drop unused Seeed library; add Panasonic FK datasheet
- U3 value TPS2553DBVR, J1/J4/J5 value L-KLS1-5416-L1-01-R
- Remove hardware/libraries/seed-xio and its fp-lib-table entry (XIAO now
  uses dock:XIAO_nRF52840_Socket_Pogo; nothing references xiao:)
- Add Panasonic FK series catalog (C13-C16, EEE-FK1E101XP)

Co-Authored-By: Claude Opus 5.5 <noreply@anthropic.com>
Parts:
- J1: value (none) -> L-KLS1-5416-L1-01-R
- U3: value (none) -> TPS2553DBVR
Changed lines of the file:
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@@
 			)
 		)
-		(property "Value" ""
+		(property "Value" "L-KLS1-5416-L1-01-R"
 			(at 38.1 81.28 0)
 			(show_name no)
@@
 			)
 		)
-		(property "Value" ""
+		(property "Value" "TPS2553DBVR"
 			(at 135.89 80.01 0)
 			(show_name no)
