File: hardware/dock/ble_base.kicad_sch (KiCad schematic)
At the start: 0 parts

Commit message: Dock schematic: review fixes, Pico 2/XIAO socket+pogo mounting
- Cross HID UART TX/RX; split ROLE_STRAP per endpoint
- VBUS sense (GP4) and USB-C CC current sensing (GP26/27) on HID endpoints
- Pogo +5V via TPS2552 enabled by DET, TPD4E1U06 ESD + 1k on pogo lines
- 2x100uF bulk on SYS_5V and keyboard VBUS; 100k EN pull-down
- Remove TPS62162 rail: XIAO from 5V, pull-ups on module 3V3 rails
- Socketed Pico 2 / XIAO footprints with P50-B1 probe holes for USB+SWD
- XIAO SWD header J8; RP2350 reset control of HID/BLE endpoints
- DESIGN.md: UART allocation, power budget, mounting, reset control
- Add .gitignore, custom libraries and datasheets

Co-Authored-By: Claude Opus 5.5 <noreply@anthropic.com>
Parts:
- added C11, C12: 1uF, Capacitor_SMD:C_0805_2012Metric_Pad1.18x1.45mm_HandSolder, symbol Device:C
- added J7: Conn_01x06, dock:Pogo-6, symbol Connector_Generic:Conn_01x06
- added J8: Conn_01x05_Pin, Connector_PinHeader_2.54mm:PinHeader_1x05_P2.54mm_Vertical, symbol Connector:Conn_01x05_Pin
- added R18: 10K, Resistor_SMD:R_0805_2012Metric_Pad1.20x1.40mm_HandSolder, symbol Device:R
- added R23: 26.1k, Resistor_SMD:R_0805_2012Metric_Pad1.20x1.40mm_HandSolder, symbol Device:R
- added R24: 10k, Resistor_SMD:R_0805_2012Metric_Pad1.20x1.40mm_HandSolder, symbol Device:R
- added R25, R26, R27, R35: 1k, Resistor_SMD:R_0805_2012Metric_Pad1.20x1.40mm_HandSolder, symbol Device:R
- added U7: XIAO_nRF52840, dock:XIAO_nRF52840_Socket_Pogo, symbol dock_custom:XIAO_nRF52840
- added U8: TPS2552DBVR, Package_TO_SOT_SMD:SOT-23-6, symbol dock_custom:TPS2552DBV
- added U9: TPD4E1U06DBVR, Package_TO_SOT_SMD:SOT-23-6, symbol dock_custom:TPD4E1U06DBV
Connections:
- new net: R23.1, U8.5 (ILIM)
- new net BLE_RST_CTRL: R35.2
- new net BLE_UART_RX: U7.7 (D6_TX_P1.11)
- new net BLE_UART_TX: U7.8 (D7_RX_P1.12)
- new net GND: C11.2, C12.2, J7.1 (Pin_1), J7.6 (Pin_6), J8.3 (Pin_3), R23.2, U7.13 (GND), U7.18 (GND), U8.2 (GND), U9.2 (GND)
- new net HOST_3V3: R24.1
- new net POGO_5V: C12.1, J7.2 (Pin_2), U8.6 (OUT), U9.1 (D1+)
- new net POGO_5V_FAULT: R24.2, U8.4 (FAULT)
- new net POGO_DET: R18.1, R27.2, U7.3 (D2_A2_P0.28), U8.3 (~{EN})
- new net POGO_DET_CONN: J7.3 (Pin_3), R27.1, U9.6 (D1-)
- new net POGO_RX: R26.2, U7.2 (D1_A1_P0.03)
- new net POGO_RX_CONN: J7.4 (Pin_4), R26.1, U9.3 (D2+)
- new net POGO_TX: R25.2, U7.1 (D0_A0_P0.02)
- new net POGO_TX_CONN: J7.5 (Pin_5), R25.1, U9.4 (D2-)
- new net SYS_5V: C11.1, U7.14 (5V_VBUS), U8.1 (IN)
- new net XIAO_3V3: J8.5 (Pin_5), R18.2, U7.12 (3V3_OUT)
- new net XIAO_RST: J8.4 (Pin_4), R35.1, U7.17 (RST)
- new net XIAO_SWCLK: J8.1 (Pin_1), U7.16 (SWCLK)
- new net XIAO_SWDIO: J8.2 (Pin_2), U7.15 (SWDIO)
- no-connect marks 0 -> 7

Commit message: Host becomes Pico 2 W (on-board BLE); remove XIAO nRF52840
- A1 -> Raspberry Pi Pico 2 W, new footprint RaspberryPi_Pico2W_Socket_Pogo
  (TP1-3 probes unchanged, SWD via 1x3 socket under the debug holes,
  TP4-6 at Pico 2 W positions, 14x9 mm antenna keep-out)
- Remove U7 (XIAO), J8 and R35; BLE UART and BLE_RST_CTRL gone
- Pogo TX/RX/DET now go to the host: GP16 (PIO TX), GP17 (PIO RX),
  GP22 (DET); R18 pulls DET up to HOST_3V3
- HID-A: CC1/CC2 on U5 and R29/R30 swapped for routing (user change)
- DESIGN.md/README/PCB_PLACEMENT.md updated; board includes in-progress
  routing and B.Cu GND zone (not yet updated from schematic)

Co-Authored-By: Claude Opus 5.5 <noreply@anthropic.com>
Parts:
- removed J8: Conn_01x05_Pin, Connector_PinHeader_2.54mm:PinHeader_1x05_P2.54mm_Vertical, symbol Connector:Conn_01x05_Pin
- removed R35: 1k, Resistor_SMD:R_0805_2012Metric_Pad1.20x1.40mm_HandSolder, symbol Device:R
- removed U7: XIAO_nRF52840, dock:XIAO_nRF52840_Socket_Pogo, symbol dock_custom:XIAO_nRF52840
Connections:
- net XIAO_3V3 is gone; now on net HOST_3V3: R18.2
- no-connect marks 7 -> 1
