File: hardware/dock/_restore_backup_2026-09-25T10-56-45-796/dock.kicad_pcb (KiCad board)
At the start: 2 copper layers, 100 x 100 mm, 69 parts, among them J1 L-KLS1-5416-L1-01-R, J2 Conn_01x05_Pin, J3 Conn_01x05_Pin, J4 L-KLS1-5416-L1-01-R, J5 L-KLS1-5416-L1-01-R, J6 Conn_01x05_Pin, J7 Conn_01x06, J8 Conn_01x05_Pin, U1 TPS2116DRL, U3 TPS2553DBVR, U4 TPD4E1U06DBVR, U5 TPD4E1U06DBVR, U6 TPD4E1U06DBVR, U7 XIAO_nRF52840, U8 TPS2552DBVR, U9 TPD4E1U06DBVR

Commit message: a small backup commit
Parts:
- moved C10 140.6 mm to (206.5, 153.5), turned to 0 degrees
- moved U6 135.2 mm to (210.5, 153.2)
- moved C15 122.7 mm to (170.7, 140.3), turned to 0 degrees
- moved C16 120.6 mm to (170.7, 148.5)
- moved R3 104.9 mm to (74.0, 153.0)
- moved C3 104.2 mm to (81.0, 156.5)
- moved J6 97.2 mm to (50.0, 149.9), turned to 0 degrees
- moved U1 96.7 mm to (80.8, 150.8), turned to 180 degrees
- moved C14 95.0 mm to (63.0, 126.5), turned to 180 degrees
- moved C9 92.6 mm to (85.5, 151.0)
- moved R2 91.0 mm to (72.0, 145.5), turned to 0 degrees
- moved C8 90.8 mm to (72.0, 142.5), turned to 180 degrees
- moved A3 90.8 mm to (216.5, 81.6)
- moved R22 90.6 mm to (213.2, 39.4), turned to 0 degrees
- moved R21 90.3 mm to (213.2, 36.4), turned to 0 degrees
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Connections:
- U5 pad 3: /HID_PERSONAL/CC2 -> /HID_PERSONAL/CC1
- U5 pad 4: /HID_PERSONAL/CC1 -> /HID_PERSONAL/CC2
Other:
- board outline removed
