File: hardware/pad/battery_charger.kicad_sch (KiCad schematic)
At the start: 0 parts

Commit message: Pad schematic: first capture (all sheets), custom symbols, hand-solder SOT-563 and MX hot-swap footprints, GPIO map
Co-Authored-By: Claude Opus 5.5 <noreply@anthropic.com>
Parts:
- added C2, C3: 10u, Capacitor_SMD:C_0805_2012Metric_Pad1.18x1.45mm_HandSolder, symbol Device:C
- added C4, C5: 100n, Capacitor_SMD:C_0805_2012Metric_Pad1.18x1.45mm_HandSolder, symbol Device:C
- added J2: NTC 10k B3950, Connector_JST:JST_XH_B2B-XH-A_1x02_P2.50mm_Vertical, symbol Connector_Generic:Conn_01x02
- added J3: Battery 2x21700 1S2P, Connector_JST:JST_XH_B2B-XH-A_1x02_P2.50mm_Vertical, symbol Connector_Generic:Conn_01x02
- added Q1, Q2: 2N7002, Package_TO_SOT_SMD:SOT-23, symbol Transistor_FET:Q_NMOS_GSD
- added Q3: FS8205A, Package_SO:TSSOP-8_4.4x3mm_P0.65mm, symbol pad_custom:FS8205A
- added R10, R11: 10k, Resistor_SMD:R_0805_2012Metric_Pad1.20x1.40mm_HandSolder, symbol Device:R
- added R12: 100, Resistor_SMD:R_0805_2012Metric_Pad1.20x1.40mm_HandSolder, symbol Device:R
- added R13: 1k, Resistor_SMD:R_0805_2012Metric_Pad1.20x1.40mm_HandSolder, symbol Device:R
- added R14, R15, R7, R8, R9: 100k, Resistor_SMD:R_0805_2012Metric_Pad1.20x1.40mm_HandSolder, symbol Device:R
- added R3: 5.6k, Resistor_SMD:R_0805_2012Metric_Pad1.20x1.40mm_HandSolder, symbol Device:R
- added R4: 75k, Resistor_SMD:R_0805_2012Metric_Pad1.20x1.40mm_HandSolder, symbol Device:R
- added R5: 8.2k, Resistor_SMD:R_0805_2012Metric_Pad1.20x1.40mm_HandSolder, symbol Device:R
- added R6: 3.3k, Resistor_SMD:R_0805_2012Metric_Pad1.20x1.40mm_HandSolder, symbol Device:R
- added U2: TP4056, Package_SO:SOIC-8-1EP_3.9x4.9mm_P1.27mm_EP2.41x3.3mm_ThermalVias, symbol Battery_Management:TP4056-42-ESOP8
- added U3: DW01A, Package_TO_SOT_SMD:SOT-23-6, symbol Battery_Management:DW01A
Connections:
- new net +3V3: R10.1, R11.1
- new net CELL_N: C4.2, J3.2 (Pin_2), Q3.2 (S1), Q3.3 (S1), U3.6 (GND)
- new net CHG_CE: Q2.3 (D), R8.2, U2.8 (CE)
- new net CHG_CHRG_N: R10.2, U2.7 (~{CHRG})
- new net CHG_FAST: Q1.1 (G), R7.1
- new net CHG_INHIBIT: Q2.1 (G), R9.1
- new net CHG_PROG: R5.1, R6.1, U2.2 (PROG)
- new net CHG_PROG_SW: Q1.3 (D), R6.2
- new net CHG_STDBY_N: R11.2, U2.6 (~{STDBY})
- new net CHG_TEMP: J2.1 (Pin_1), R3.2, R4.1, U2.1 (TEMP)
- new net DW_CS: R13.1, U3.2 (CS)
- new net DW_OC: Q3.5 (G2), U3.3 (OC)
- new net DW_OD: Q3.4 (G1), U3.1 (OD)
- new net DW_VCC: C4.1, R12.2, U3.5 (VCC)
- new net FET_D12: Q3.1 (D12), Q3.8 (D12)
- new net GND: C2.2, C3.2, C5.2, J2.2 (Pin_2), Q1.2 (S), Q2.2 (S), Q3.6 (S2), Q3.7 (S2), R13.2, R15.2, R4.2, R5.2, R7.2, R9.2, U2.3 (GND), U2.9 (EPAD)
- new net POGO_5V: C2.1, R3.1, R8.1, U2.4 (V_{CC})
- new net VBAT: C3.1, J3.1 (Pin_1), R12.1, R14.1, U2.5 (BAT)
- new net VBAT_SENSE: C5.1, R14.2, R15.1
Other:
- note added: "CE defaults high (charging on) through 100k from POGO_5V; CHG_INHIBIT high pulls CE low (Pico holds the docked 3.90-4.00 V window)."
- note added: "CELL_N = cell negative (DW01A ground). GND = pack negative = board ground."
- note added: "Cell protection DW01A + FS8205A in the negative lead: over-discharge 2.40 V, overcharge 4.30 V, overcurrent 150 mV / (2 x 25 mOhm) = about 3 A."
- note added: "Li-ion charger TP4056: 4.2 V CC-CV. I = 1200 / R_PROG. 8.2k alone = 146 mA (slow); Q with CHG_FAST high adds 3.3k in parallel = 510 mA (fast)."
- note added: "TEMP window 45-80 % of VCC: R 5.6k to VCC, NTC 10k B3950 parallel 75k to GND = charge only between about 0 and 45 C."
- note added: "VBAT_SENSE = VBAT / 2 to Pico ADC0 (GP26). Permanent divider, about 18 uA."
