File: hardware/pad/battery_charger.kicad_sch (KiCad schematic)
At the start: 24 parts, among them J2 NTC 10k B3950, J3 Battery 2x21700 1S2P, Q1 2N7002, Q2 2N7002, Q3 FS8205A, U2 TP4056, U3 DW01A

Commit message: Pad PCB: first placement; SWD header removed, side-entry JST connectors, new footprints
- J4 (SWD) removed; A1 on the NoSWD Pico socket footprint (holes would sit under key 5)
- J1/J7/J2/J3 side-entry JST (S*B), J5 stays vertical
- New footprints: PEC11R encoder (13.2 mm lugs), SOIC-8-1EP hand-solder (TP4056),
  narrower SOT-563 pads
- All footprints placed on the 100 x 92 board; ring LEDs radial at R 12.7,
  encoders at 16.6 / 83.4; edge clearance rule 0.2 mm
- PCB_PLACEMENT.md and placement drawings in docs/

Co-Authored-By: Claude Opus 5.5 <noreply@anthropic.com>
Parts:
- J2, J3: footprint Connector_JST:JST_XH_B2B-XH-A_1x02_P2.50mm_Vertical -> Connector_JST:JST_XH_S2B-XH-A_1x02_P2.50mm_Horizontal
- U2: footprint Package_SO:SOIC-8-1EP_3.9x4.9mm_P1.27mm_EP2.41x3.3mm_ThermalVias -> dock:SOIC-8-1EP_3.9x4.9mm_HandSolder
Changed lines of the file:
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@@
 			)
 		)
-		(property "Footprint" "Package_SO:SOIC-8-1EP_3.9x4.9mm_P1.27mm_EP2.41x3.3mm_ThermalVias"
+		(property "Footprint" "dock:SOIC-8-1EP_3.9x4.9mm_HandSolder"
 			(at 88.9 78.74 0)
 			(hide yes)
@@
 			)
 		)
-		(property "Footprint" "Connector_JST:JST_XH_B2B-XH-A_1x02_P2.50mm_Vertical"
+		(property "Footprint" "Connector_JST:JST_XH_S2B-XH-A_1x02_P2.50mm_Horizontal"
 			(at 154.94 50.8 0)
 			(hide yes)
@@
 			)
 		)
-		(property "Footprint" "Connector_JST:JST_XH_B2B-XH-A_1x02_P2.50mm_Vertical"
+		(property "Footprint" "Connector_JST:JST_XH_S2B-XH-A_1x02_P2.50mm_Horizontal"
 			(at 148.59 76.2 0)
 			(hide yes)
