File: hardware/pad/display.kicad_sch (KiCad schematic)
At the start: 0 parts

Commit message: Pad schematic: first capture (all sheets), custom symbols, hand-solder SOT-563 and MX hot-swap footprints, GPIO map
Co-Authored-By: Claude Opus 5.5 <noreply@anthropic.com>
Parts:
- added C54, C55: 1u, Capacitor_SMD:C_0805_2012Metric_Pad1.18x1.45mm_HandSolder, symbol Device:C
- added J6: OLED 1.3in SPI, Connector_PinSocket_2.54mm:PinSocket_1x07_P2.54mm_Vertical, symbol Connector_Generic:Conn_01x07
- added R30: 100k, Resistor_SMD:R_0805_2012Metric_Pad1.20x1.40mm_HandSolder, symbol Device:R
- added R31: 100, Resistor_SMD:R_0805_2012Metric_Pad1.20x1.40mm_HandSolder, symbol Device:R
- added U8: TPS22919DCK, Package_TO_SOT_SMD:SOT-363_SC-70-6, symbol Power_Management:TPS22919DCK
Connections:
- new net +3V3: C54.1, U8.1 (IN)
- new net GND: C54.2, C55.2, J6.1 (Pin_1), R30.2, U8.2 (GND)
- new net OLED_CS: J6.7 (Pin_7)
- new net OLED_DC: J6.6 (Pin_6)
- new net OLED_EN: R30.1, U8.3 (ON)
- new net OLED_MOSI: J6.4 (Pin_4)
- new net OLED_QOD: R31.2, U8.5 (QOD)
- new net OLED_RES: J6.5 (Pin_5)
- new net OLED_SCK: J6.3 (Pin_3)
- new net OLED_VCC: C55.1, J6.2 (Pin_2), R31.1, U8.6 (OUT)
Other:
- note added: "1.3 inch 128x64 SPI OLED (SH1106 or SSD1306, chosen in firmware). Pin order on the module: GND VCC SCK SDA(MOSI) RES DC CS."
- note added: "TPS22919 switches +3V3 to the module (OLED_EN from the Pico, 100k pull-down = off at boot). QOD to OUT through 100R = controlled quick discharge when off (datasheet option)."
