File: hardware/pad/dock_interface.kicad_sch (KiCad schematic)
At the start: 0 parts

Commit message: Pad schematic: first capture (all sheets), custom symbols, hand-solder SOT-563 and MX hot-swap footprints, GPIO map
Co-Authored-By: Claude Opus 5.5 <noreply@anthropic.com>
Parts:
- added C1: 10u, Capacitor_SMD:C_0805_2012Metric_Pad1.18x1.45mm_HandSolder, symbol Device:C
- added D1: SMAJ5.0A, Diode_SMD:D_SMA, symbol Device:D_Zener
- added J1: Pogo_6p, dock:Pogo-6, symbol Connector_Generic:Conn_01x06
- added R1, R2: 1k, Resistor_SMD:R_0805_2012Metric_Pad1.20x1.40mm_HandSolder, symbol Device:R
- added U1: TPD4E1U06DBVR, Package_TO_SOT_SMD:SOT-23-6, symbol pad_custom:TPD4E1U06DBV
Connections:
- new net GND: C1.2, D1.2 (A), J1.1 (Pin_1), J1.4 (Pin_4), J1.6 (Pin_6), U1.2 (GND)
- new net PAD_UART_RX: R1.2
- new net PAD_UART_TX: R2.1
- new net POGO_5V: C1.1, D1.1 (K), J1.5 (Pin_5)
- new net POGO_DRX: J1.3 (Pin_3), R2.2, U1.3 (D2+)
- new net POGO_DTX: J1.2 (Pin_2), R1.1, U1.1 (D1+)
- no-connect marks 0 -> 3
Other:
- note added: "1k series on both sides: 2k total when docked (about 40 ns edge, fine at 1 Mbaud)."
- note added: "POGO_DTX = dock TX contact (pad receives), POGO_DRX = dock RX contact (pad transmits). DET is tied to GND: that enables the dock TPS2552."
- note added: "Pogo contacts, pad side. Face-to-face mating mirrors the dock order (dock: GND | +5V | DET | RX | TX | GND)."
- note added: "Undocked, a bridge from +5V to RX/TX injects at most about 1.4 mA into the pad Pico."
