File: hardware/pad/inputs.kicad_sch (KiCad schematic)
At the start: 0 parts

Commit message: Pad schematic: first capture (all sheets), custom symbols, hand-solder SOT-563 and MX hot-swap footprints, GPIO map
Co-Authored-By: Claude Opus 5.5 <noreply@anthropic.com>
Parts:
- added C12: 100n, Capacitor_SMD:C_0805_2012Metric_Pad1.18x1.45mm_HandSolder, symbol Device:C
- added C13, C14, C15, C16: 10n, Capacitor_SMD:C_0805_2012Metric_Pad1.18x1.45mm_HandSolder, symbol Device:C
- added J5: Selector ON-OFF-ON, Connector_JST:JST_XH_B3B-XH-A_1x03_P2.50mm_Vertical, symbol Connector_Generic:Conn_01x03
- added R22, R23: 4.7k, Resistor_SMD:R_0805_2012Metric_Pad1.20x1.40mm_HandSolder, symbol Device:R
- added R24, R25, R26, R27, R28: 10k, Resistor_SMD:R_0805_2012Metric_Pad1.20x1.40mm_HandSolder, symbol Device:R
- added SW1, SW10, SW11, SW12, SW2, SW3, SW4, SW5, SW6, SW7, SW8, SW9: Razer Yellow (MX, hot-swap), dock:SW_MX_Hotswap_Kailh, symbol Switch:SW_Push
- added SW13, SW14: PEC11R-4220F-S0024, Rotary_Encoder:RotaryEncoder_Alps_EC11E-Switch_Vertical_H20mm, symbol Device:RotaryEncoder_Switch
- added U6: TCA9555PWR, Package_SO:TSSOP-24_4.4x7.8mm_P0.65mm, symbol Interface_Expansion:TCA9555PWR
Connections:
- new net +3V3: C12.1, R22.1, R23.1, R24.1, R25.1, R26.1, R27.1, R28.1, U6.24 (VCC)
- new net ENC1_A: C13.1, R25.2, SW13.A
- new net ENC1_B: C14.1, R26.2, SW13.B
- new net ENC1_SW: SW13.S1, U6.17 (P14)
- new net ENC2_A: C15.1, R27.2, SW14.A
- new net ENC2_B: C16.1, R28.2, SW14.B
- new net ENC2_SW: SW14.S1, U6.18 (P15)
- new net GND: C12.2, C13.2, C14.2, C15.2, C16.2, J5.2 (Pin_2), SW1.2, SW10.2, SW11.2, SW12.2, SW13.C, SW13.S2, SW14.C, SW14.S2, SW2.2, SW3.2, SW4.2, SW5.2, SW6.2, SW7.2, SW8.2, SW9.2, U6.12 (GND), U6.2 (A1), U6.21 (A0), U6.3 (A2)
- new net I2C_SCL: R23.2, U6.22 (SCL)
- new net I2C_SDA: R22.2, U6.23 (SDA)
- new net KEY1: SW1.1, U6.4 (P00)
- new net KEY10: SW10.1, U6.14 (P11)
- new net KEY11: SW11.1, U6.15 (P12)
- new net KEY12: SW12.1, U6.16 (P13)
- new net KEY2: SW2.1, U6.5 (P01)
- new net KEY3: SW3.1, U6.6 (P02)
- new net KEY4: SW4.1, U6.7 (P03)
- new net KEY5: SW5.1, U6.8 (P04)
- new net KEY6: SW6.1, U6.9 (P05)
- new net KEY7: SW7.1, U6.10 (P06)
- new net KEY8: SW8.1, U6.11 (P07)
- new net KEY9: SW9.1, U6.13 (P10)
- new net SEL_A: J5.1 (Pin_1), U6.19 (P16)
- new net SEL_B: J5.3 (Pin_3), U6.20 (P17)
- new net TCA_INT_N: R24.2, U6.1 (~{INT})
Other:
- note added: "Encoder A/B: 10k pull-up + 10 nF to GND (debounce), decoded by Pico PIO. Common (C) to GND."
- note added: "P00-P13 = KEY1-KEY12, P14/P15 = encoder push, P16/P17 = PERSONAL/OFF/WORK selector (A/B, see DESIGN.md 8.3)."
- note added: "Panel toggle: common to pin 2 (GND), PERSONAL throw to pin 1 (SEL_A), WORK throw to pin 3 (SEL_B)."
- note added: "TCA9555 (address 0x20). Its ports have internal 100k pull-ups, so keys and switches go straight to GND (active low)."
