File: hardware/pad/inputs.kicad_sch (KiCad schematic)
At the start: 28 parts, among them J5 Selector ON-OFF-ON, SW1 Razer Yellow (MX, hot-swap), SW10 Razer Yellow (MX, hot-swap), SW11 Razer Yellow (MX, hot-swap), SW12 Razer Yellow (MX, hot-swap), SW13 PEC11R-4220F-S0024, SW14 PEC11R-4220F-S0024, SW2 Razer Yellow (MX, hot-swap), SW3 Razer Yellow (MX, hot-swap), SW4 Razer Yellow (MX, hot-swap), SW5 Razer Yellow (MX, hot-swap), SW6 Razer Yellow (MX, hot-swap), SW7 Razer Yellow (MX, hot-swap), SW8 Razer Yellow (MX, hot-swap), SW9 Razer Yellow (MX, hot-swap), U6 TCA9555PWR

Commit message: Pad PCB: first placement; SWD header removed, side-entry JST connectors, new footprints
- J4 (SWD) removed; A1 on the NoSWD Pico socket footprint (holes would sit under key 5)
- J1/J7/J2/J3 side-entry JST (S*B), J5 stays vertical
- New footprints: PEC11R encoder (13.2 mm lugs), SOIC-8-1EP hand-solder (TP4056),
  narrower SOT-563 pads
- All footprints placed on the 100 x 92 board; ring LEDs radial at R 12.7,
  encoders at 16.6 / 83.4; edge clearance rule 0.2 mm
- PCB_PLACEMENT.md and placement drawings in docs/

Co-Authored-By: Claude Opus 5.5 <noreply@anthropic.com>
Parts:
- SW13, SW14: footprint Rotary_Encoder:RotaryEncoder_Alps_EC11E-Switch_Vertical_H20mm -> dock:RotaryEncoder_Bourns_PEC11R-4xxxF-S_Vertical
Changed lines of the file:
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@@
 			)
 		)
-		(property "Footprint" "Rotary_Encoder:RotaryEncoder_Alps_EC11E-Switch_Vertical_H20mm"
+		(property "Footprint" "dock:RotaryEncoder_Bourns_PEC11R-4xxxF-S_Vertical"
 			(at 73.66 157.48 0)
 			(hide yes)
@@
 			)
 		)
-		(property "Footprint" "Rotary_Encoder:RotaryEncoder_Alps_EC11E-Switch_Vertical_H20mm"
+		(property "Footprint" "dock:RotaryEncoder_Bourns_PEC11R-4xxxF-S_Vertical"
 			(at 127 157.48 0)
 			(hide yes)
