File: hardware/pad/pad.kicad_sch (KiCad schematic)
At the start: 0 parts

Commit message: Pad schematic: first capture (all sheets), custom symbols, hand-solder SOT-563 and MX hot-swap footprints, GPIO map
Co-Authored-By: Claude Opus 5.5 <noreply@anthropic.com>
Other:
- sheet NRF52840 renamed MCU
- sheet MCU: file nrf52840.kicad_sch -> mcu.kicad_sch
