File: hardware/pad/power_rails.kicad_sch (KiCad schematic)
At the start: 0 parts

Commit message: Pad schematic: first capture (all sheets), custom symbols, hand-solder SOT-563 and MX hot-swap footprints, GPIO map
Co-Authored-By: Claude Opus 5.5 <noreply@anthropic.com>
Parts:
- added C10, C11: 22u, Capacitor_SMD:C_1206_3216Metric_Pad1.33x1.80mm_HandSolder, symbol Device:C
- added C6: 1u, Capacitor_SMD:C_0805_2012Metric_Pad1.18x1.45mm_HandSolder, symbol Device:C
- added C7, C8: 10u, Capacitor_SMD:C_0805_2012Metric_Pad1.18x1.45mm_HandSolder, symbol Device:C
- added C9: 10u, Capacitor_SMD:C_1206_3216Metric_Pad1.33x1.80mm_HandSolder, symbol Device:C
- added L1: 1u, Inductor_SMD:L_Coilcraft_XxL4030, symbol Device:L
- added R16: 300k, Resistor_SMD:R_0805_2012Metric_Pad1.20x1.40mm_HandSolder, symbol Device:R
- added R17, R19, R21: 100k, Resistor_SMD:R_0805_2012Metric_Pad1.20x1.40mm_HandSolder, symbol Device:R
- added R18: 10k, Resistor_SMD:R_0805_2012Metric_Pad1.20x1.40mm_HandSolder, symbol Device:R
- added R20: 750k, Resistor_SMD:R_0805_2012Metric_Pad1.20x1.40mm_HandSolder, symbol Device:R
- added U4: TPS2116DRL, dock:SOT-583-8_HandSolder, symbol Power_Management:TPS2116DRL
- added U5: TPS61023DRLR, dock:SOT-563-6_HandSolder, symbol pad_custom:TPS61023DRL
Connections:
- new net +3V3: R18.1
- new net 5V_RGB: C10.1, C11.1, R20.1, U5.6 (VOUT)
- new net BOOST_FB: R20.2, R21.1, U5.1 (FB)
- new net BOOST_SW: L1.2, U5.5 (SW)
- new net DOCKED: R18.2, U4.8 (ST)
- new net GND: C10.2, C11.2, C6.2, C7.2, C8.2, C9.2, R17.2, R19.2, R21.2, U4.1 (GND), U5.4 (GND)
- new net MUX_PR1: R16.2, R17.1, U4.4 (PR1)
- new net PAD_SYS: C7.1, C8.1, C9.1, L1.1, U4.2 (VOUT), U4.7 (VOUT), U5.3 (VIN)
- new net POGO_5V: R16.1, U4.3 (VIN1), U4.5 (MODE)
- new net RGB_EN: R19.1, U5.2 (EN)
- new net VBAT: C6.1, U4.6 (VIN2)
Other:
- note added: "L: 1 uH shielded 4x4 mm, Isat >= 4.5 A, DCR <= 20 mOhm (Wurth 74438357010 / Coilcraft XEL4030-102ME)."
- note added: "ST is high while VIN1 (pogo) is in use: DOCKED to the Pico. Reverse-current blocking keeps Pico USB VBUS out of the cell."
- note added: "TPS2116 power path: POGO_5V (VIN1, priority) or VBAT (VIN2) to PAD_SYS. PR1 300k/100k = switchover at about 4.0 V; MODE tied to VIN1 (as on the dock)."
- note added: "TPS61023 boost: PAD_SYS to 5V_RGB. VOUT = 0.6 V x (1 + 750k/100k) = about 5.05 V. Pass-through when docked."
