File: hardware/pad/rgb.kicad_sch (KiCad schematic)
At the start: 0 parts

Commit message: Pad schematic: first capture (all sheets), custom symbols, hand-solder SOT-563 and MX hot-swap footprints, GPIO map
Co-Authored-By: Claude Opus 5.5 <noreply@anthropic.com>
Parts:
- added C17, C18, C19, C20, C21, C22, C23, C24, C25, C26, C27, C28, C29, C30, C31, C32, C33, C34, C35, C36, C37, C38, C39, C40, C41, C42, C43, C44, C45, C46, C47, C48, C49, C50, C51, C52, C53: 100n, Capacitor_SMD:C_0805_2012Metric_Pad1.18x1.45mm_HandSolder, symbol Device:C
- added D10, D11, D12, D13, D14, D15, D16, D17, D18, D19, D2, D20, D21, D22, D23, D24, D25, D26, D27, D28, D29, D3, D30, D31, D32, D33, D34, D35, D36, D37, D4, D5, D6, D7, D8, D9: SK6812MINI-E, LED_SMD:LED_SK6812MINI-E_3.2x2.8mm_P1.5mm_ReverseMount, symbol LED:SK6812MINI-E
- added R29: 47, Resistor_SMD:R_0805_2012Metric_Pad1.20x1.40mm_HandSolder, symbol Device:R
- added U7: 74AHCT1G125, Package_TO_SOT_SMD:SOT-23-5, symbol 74xGxx:74AHCT1G125
Connections:
- new net 5V_RGB: C17.1, C18.1, C19.1, C20.1, C21.1, C22.1, C23.1, C24.1, C25.1, C26.1, C27.1, C28.1, C29.1, C30.1, C31.1, C32.1, C33.1, C34.1, C35.1, C36.1, C37.1, C38.1, C39.1, C40.1, C41.1, C42.1, C43.1, C44.1, C45.1, C46.1, C47.1, C48.1, C49.1, C50.1, C51.1, C52.1, C53.1, D10.3 (VDD), D11.3 (VDD), D12.3 (VDD), D13.3 (VDD), D14.3 (VDD), D15.3 (VDD), D16.3 (VDD), D17.3 (VDD), D18.3 (VDD), D19.3 (VDD), D2.3 (VDD), D20.3 (VDD), D21.3 (VDD), D22.3 (VDD), D23.3 (VDD), D24.3 (VDD), D25.3 (VDD), D26.3 (VDD), D27.3 (VDD), D28.3 (VDD), D29.3 (VDD), D3.3 (VDD), D30.3 (VDD), D31.3 (VDD), D32.3 (VDD), D33.3 (VDD), D34.3 (VDD), D35.3 (VDD), D36.3 (VDD), D37.3 (VDD), D4.3 (VDD), D5.3 (VDD), D6.3 (VDD), D7.3 (VDD), D8.3 (VDD), D9.3 (VDD), U7.5 (VCC)
- new net GND: C17.2, C18.2, C19.2, C20.2, C21.2, C22.2, C23.2, C24.2, C25.2, C26.2, C27.2, C28.2, C29.2, C30.2, C31.2, C32.2, C33.2, C34.2, C35.2, C36.2, C37.2, C38.2, C39.2, C40.2, C41.2, C42.2, C43.2, C44.2, C45.2, C46.2, C47.2, C48.2, C49.2, C50.2, C51.2, C52.2, C53.2, D10.1 (VSS), D11.1 (VSS), D12.1 (VSS), D13.1 (VSS), D14.1 (VSS), D15.1 (VSS), D16.1 (VSS), D17.1 (VSS), D18.1 (VSS), D19.1 (VSS), D2.1 (VSS), D20.1 (VSS), D21.1 (VSS), D22.1 (VSS), D23.1 (VSS), D24.1 (VSS), D25.1 (VSS), D26.1 (VSS), D27.1 (VSS), D28.1 (VSS), D29.1 (VSS), D3.1 (VSS), D30.1 (VSS), D31.1 (VSS), D32.1 (VSS), D33.1 (VSS), D34.1 (VSS), D35.1 (VSS), D36.1 (VSS), D37.1 (VSS), D4.1 (VSS), D5.1 (VSS), D6.1 (VSS), D7.1 (VSS), D8.1 (VSS), D9.1 (VSS), U7.1, U7.3 (GND)
- new net LED_DIN1: D2.2 (DIN), R29.2
- new net LED_DIN10: D10.4 (DOUT), D11.2 (DIN)
- new net LED_DIN11: D11.4 (DOUT), D12.2 (DIN)
- new net LED_DIN12: D12.4 (DOUT), D13.2 (DIN)
- new net LED_DIN13: D13.4 (DOUT), D14.2 (DIN)
- new net LED_DIN14: D14.4 (DOUT), D15.2 (DIN)
- new net LED_DIN15: D15.4 (DOUT), D16.2 (DIN)
- new net LED_DIN16: D16.4 (DOUT), D17.2 (DIN)
- new net LED_DIN17: D17.4 (DOUT), D18.2 (DIN)
- new net LED_DIN18: D18.4 (DOUT), D19.2 (DIN)
- new net LED_DIN19: D19.4 (DOUT), D20.2 (DIN)
- new net LED_DIN2: D2.4 (DOUT), D3.2 (DIN)
- new net LED_DIN20: D20.4 (DOUT), D21.2 (DIN)
- new net LED_DIN21: D21.4 (DOUT), D22.2 (DIN)
- new net LED_DIN22: D22.4 (DOUT), D23.2 (DIN)
- new net LED_DIN23: D23.4 (DOUT), D24.2 (DIN)
- new net LED_DIN24: D24.4 (DOUT), D25.2 (DIN)
- new net LED_DIN25: D25.4 (DOUT), D26.2 (DIN)
- new net LED_DIN26: D26.4 (DOUT), D27.2 (DIN)
- new net LED_DIN27: D27.4 (DOUT), D28.2 (DIN)
- new net LED_DIN28: D28.4 (DOUT), D29.2 (DIN)
- new net LED_DIN29: D29.4 (DOUT), D30.2 (DIN)
- new net LED_DIN3: D3.4 (DOUT), D4.2 (DIN)
- new net LED_DIN30: D30.4 (DOUT), D31.2 (DIN)
- new net LED_DIN31: D31.4 (DOUT), D32.2 (DIN)
- new net LED_DIN32: D32.4 (DOUT), D33.2 (DIN)
- new net LED_DIN33: D33.4 (DOUT), D34.2 (DIN)
- new net LED_DIN34: D34.4 (DOUT), D35.2 (DIN)
- new net LED_DIN35: D35.4 (DOUT), D36.2 (DIN)
- new net LED_DIN36: D36.4 (DOUT), D37.2 (DIN)
- new net LED_DIN4: D4.4 (DOUT), D5.2 (DIN)
- new net LED_DIN5: D5.4 (DOUT), D6.2 (DIN)
- new net LED_DIN6: D6.4 (DOUT), D7.2 (DIN)
- new net LED_DIN7: D7.4 (DOUT), D8.2 (DIN)
- new net LED_DIN8: D8.4 (DOUT), D9.2 (DIN)
- new net LED_DIN9: D10.2 (DIN), D9.4 (DOUT)
- new net RGB_BUF: R29.1, U7.4
- new net RGB_DATA_3V3: U7.2
- no-connect marks 0 -> 1
Other:
- note added: "36 x SK6812MINI-E on 5V_RGB, one chain. Order to be fixed at layout (keys 1-12, ring 1, ring 2). 100 nF per LED."
- note added: "Data: Pico 3.3 V (PIO) through SN74AHCT1G125 (VCC = 5V_RGB, so data drive dies with the rail) and a 47R series resistor."
