File: hardware/pad/rgb.kicad_sch (KiCad schematic)
At the start: 75 parts, among them U7 74AHCT1G125

Commit message: Pad schematic: hand-redrawn from the connection guide; netlist verified against the reference
Connections:
- net LED_DIN24 is gone; now on net LED_DIN2: D24.4 (DOUT), D25.2 (DIN)
- net LED_DIN2: no longer D2.4 (DOUT), D3.2 (DIN)
- net LED_DIN10: no longer names the net of D10.4 (DOUT), D11.2 (DIN)
- net LED_DIN11: no longer names the net of D11.4 (DOUT), D12.2 (DIN)
- net LED_DIN12: no longer names the net of D12.4 (DOUT), D13.2 (DIN)
- net LED_DIN13: no longer names the net of D13.4 (DOUT), D14.2 (DIN)
- net LED_DIN14: no longer names the net of D14.4 (DOUT), D15.2 (DIN)
- net LED_DIN15: no longer names the net of D15.4 (DOUT), D16.2 (DIN)
- net LED_DIN16: no longer names the net of D16.4 (DOUT), D17.2 (DIN)
- net LED_DIN17: no longer names the net of D17.4 (DOUT), D18.2 (DIN)
- net LED_DIN18: no longer names the net of D18.4 (DOUT), D19.2 (DIN)
- net LED_DIN19: no longer names the net of D19.4 (DOUT), D20.2 (DIN)
- net LED_DIN20: no longer names the net of D20.4 (DOUT), D21.2 (DIN)
- net LED_DIN21: no longer names the net of D21.4 (DOUT), D22.2 (DIN)
- net LED_DIN22: no longer names the net of D22.4 (DOUT), D23.2 (DIN)
- net LED_DIN23: no longer names the net of D23.4 (DOUT), D24.2 (DIN)
- net LED_DIN25: no longer names the net of D25.4 (DOUT), D26.2 (DIN)
- net LED_DIN26: no longer names the net of D26.4 (DOUT), D27.2 (DIN)
- net LED_DIN27: no longer names the net of D27.4 (DOUT), D28.2 (DIN)
- net LED_DIN28: no longer names the net of D28.4 (DOUT), D29.2 (DIN)
- net LED_DIN29: no longer names the net of D29.4 (DOUT), D30.2 (DIN)
- net LED_DIN3: no longer names the net of D3.4 (DOUT), D4.2 (DIN)
- net LED_DIN30: no longer names the net of D30.4 (DOUT), D31.2 (DIN)
- net LED_DIN31: no longer names the net of D31.4 (DOUT), D32.2 (DIN)
- net LED_DIN32: no longer names the net of D32.4 (DOUT), D33.2 (DIN)
- net LED_DIN33: no longer names the net of D33.4 (DOUT), D34.2 (DIN)
- net LED_DIN34: no longer names the net of D34.4 (DOUT), D35.2 (DIN)
- net LED_DIN35: no longer names the net of D35.4 (DOUT), D36.2 (DIN)
- net LED_DIN36: no longer names the net of D36.4 (DOUT), D37.2 (DIN)
- net LED_DIN4: no longer names the net of D4.4 (DOUT), D5.2 (DIN)
- net LED_DIN5: no longer names the net of D5.4 (DOUT), D6.2 (DIN)
- net LED_DIN6: no longer names the net of D6.4 (DOUT), D7.2 (DIN)
- net LED_DIN7: no longer names the net of D7.4 (DOUT), D8.2 (DIN)
- net LED_DIN8: no longer names the net of D8.4 (DOUT), D9.2 (DIN)
- net LED_DIN9: no longer names the net of D10.2 (DIN), D9.4 (DOUT)
- net RGB_BUF: no longer names the net of R29.1, U7.4
- new net: D2.4 (DOUT), D3.2 (DIN)
