File: hardware/pad/mcu.kicad_sch (KiCad schematic)
At the start: 2 parts, among them J4 SWD

Commit message: Pad: connection and placement guide, probe-free Pico 2 W socket footprint
Co-Authored-By: Claude Opus 5.5 <noreply@anthropic.com>
Parts:
- A1: footprint dock:RaspberryPi_Pico2W_Socket_Pogo -> dock:RaspberryPi_Pico2W_Socket
Changed lines of the file:
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@@
 			)
 		)
-		(property "Footprint" "dock:RaspberryPi_Pico2W_Socket_Pogo"
+		(property "Footprint" "dock:RaspberryPi_Pico2W_Socket"
 			(at 119.38 99.06 0)
 			(hide yes)
