File: hardware/dock-v2/mcu_a.kicad_sch (KiCad schematic)
At the start: 0 parts

Commit message: Dock v2: all parts placed on their sheets (not wired)
149 parts across POWER, USB_PORTS, MCU_A, MCU_B, BLE and POGO (A3), in
labelled groups, with references (sheet x 100), values, footprints, LCSC
numbers (hidden LCSC field) and a Note per part. Only unconnected-pin ERC
messages remain.

5 V buck values from TI's TPS54331 Table 7-1 (5 V design), moved to Basic
parts: 12k/2.2k feedback (5.16 V), 51k + 4.7nF + 47pF compensation, 10 nF
soft start, 3 x 22 uF out; recorded in docs/dock-v2-power-input.md.
New footprint dock_v2:CP_Radial_D6.3mm_P5.00mm for the hand-soldered 220 uF.

Co-Authored-By: Claude Opus 5.5 <noreply@anthropic.com>
Parts:
- added C301, C302: 4.7uF, dock_v2:C_0402_RPi_Wide, symbol Device:C
- added C303: 4.7uF, Capacitor_SMD:C_0402_1005Metric, symbol Device:C
- added C304, C305, C306, C307, C308, C309, C310, C311, C312, C313: 100nF, Capacitor_SMD:C_0402_1005Metric, symbol Device:C
- added C314: 10uF, Capacitor_SMD:C_0805_2012Metric, symbol Device:C
- added C315, C316: 15pF, Capacitor_SMD:C_0402_1005Metric, symbol Device:C
- added D301: LED red, LED_SMD:LED_0603_1608Metric, symbol Device:LED
- added L301: 3.3uH, dock_v2:L_Abracon_AOTA-B201610S3R3_0806, symbol Device:L
- added R301: 33, Resistor_SMD:R_0402_1005Metric, symbol Device:R
- added R302, R303, R305: 1k, Resistor_SMD:R_0402_1005Metric, symbol Device:R
- added SW301, SW302: SW_Push, Button_Switch_SMD:SW_Push_1P1T_XKB_TS-1187A, symbol Switch:SW_Push
- added TP301, TP302, TP303: TestPoint, TestPoint:TestPoint_Pad_D1.0mm, symbol Connector:TestPoint
- added U301: RP2354A, dock_v2:RP2350A_QFN-60_RPi_Vias, symbol dock_v2_custom:RP2354A_RPiFP
- added Y301: 12MHz, Crystal:Crystal_SMD_3225-4Pin_3.2x2.5mm, symbol Device:Crystal_GND24
Connections:
- new net: U301.1 (IOVDD), U301.11 (IOVDD), U301.20 (IOVDD), U301.30 (IOVDD), U301.38 (IOVDD), U301.45 (IOVDD)
- new net: U301.23 (DVDD), U301.39 (DVDD), U301.6 (DVDD)
- new net: Y301.2 (G), Y301.4 (G)
Other:
- note added: "Buttons, SWD pads, LED"
- note added: "Core regulator (copy_rpi_core_layout.py)"
- note added: "Crystal"
- note added: "Decoupling"
- note added: "RP2354A A"
