File: hardware/dock-v2/usb_ports.kicad_sch (KiCad schematic)
At the start: 0 parts

Commit message: Dock v2: all parts placed on their sheets (not wired)
149 parts across POWER, USB_PORTS, MCU_A, MCU_B, BLE and POGO (A3), in
labelled groups, with references (sheet x 100), values, footprints, LCSC
numbers (hidden LCSC field) and a Note per part. Only unconnected-pin ERC
messages remain.

5 V buck values from TI's TPS54331 Table 7-1 (5 V design), moved to Basic
parts: 12k/2.2k feedback (5.16 V), 51k + 4.7nF + 47pF compensation, 10 nF
soft start, 3 x 22 uF out; recorded in docs/dock-v2-power-input.md.
New footprint dock_v2:CP_Radial_D6.3mm_P5.00mm for the hand-soldered 220 uF.

Co-Authored-By: Claude Opus 5.5 <noreply@anthropic.com>
Parts:
- added C201: 220uF 16V, dock_v2:CP_Radial_D6.3mm_P5.00mm, symbol Device:C_Polarized
- added C202: 10uF, Capacitor_SMD:C_0805_2012Metric, symbol Device:C
- added C203, C204: 1uF, Capacitor_SMD:C_0402_1005Metric, symbol Device:C
- added J201, J202, J203: TYPE-C-31-M-12, Connector_USB:USB_C_Receptacle_HRO_TYPE-C-31-M-12, symbol Connector:USB_C_Receptacle_USB2.0_16P
- added R201, R202, R214, R220: 33k, Resistor_SMD:R_0402_1005Metric, symbol Device:R
- added R203, R204, R210: 15k, Resistor_SMD:R_0402_1005Metric, symbol Device:R
- added R205, R206, R215, R216, R221, R222: 22, Resistor_SMD:R_0402_1005Metric, symbol Device:R
- added R207: 6.8k, Resistor_SMD:R_0402_1005Metric, symbol Device:R
- added R208: 100k, Resistor_SMD:R_0402_1005Metric, symbol Device:R
- added R209: 10k, Resistor_SMD:R_0402_1005Metric, symbol Device:R
- added R211, R212, R217, R218: 5.1k, Resistor_SMD:R_0402_1005Metric, symbol Device:R
- added R213, R219: 22k, Resistor_SMD:R_0402_1005Metric, symbol Device:R
- added U201, U203, U204: TPD4E1U06DBVR, Package_TO_SOT_SMD:SOT-23-6, symbol dock_v2_custom:TPD4E1U06DBV
- added U202: SY6280AAC, Package_TO_SOT_SMD:SOT-23-5, symbol dock_v2_custom:SY6280AAC
Connections:
- new net: J201.A1 (GND), J201.A12 (GND), J201.B1 (GND), J201.B12 (GND)
- new net: J201.A4 (VBUS), J201.A9 (VBUS), J201.B4 (VBUS), J201.B9 (VBUS)
- new net: J203.A1 (GND), J203.A12 (GND), J203.B1 (GND), J203.B12 (GND)
- new net: J203.A4 (VBUS), J203.A9 (VBUS), J203.B4 (VBUS), J203.B9 (VBUS)
- new net: J202.A1 (GND), J202.A12 (GND), J202.B1 (GND), J202.B12 (GND)
- new net: J202.A4 (VBUS), J202.A9 (VBUS), J202.B4 (VBUS), J202.B9 (VBUS)
Other:
- note added: "Keyboard VBUS switch"
- note added: "Keyboard port J201 (USB-C source, left edge)"
- note added: "Personal PC port J202 (back, left)"
- note added: "Work PC port J203 (back, right)"
