File: hardware/dock-v2/usb_ports.kicad_sch (KiCad schematic)
At the start: 33 parts, among them J201 TYPE-C-31-M-12, J202 TYPE-C-31-M-12, J203 TYPE-C-31-M-12, U201 TPD4E1U06DBVR, U202 SY6280AAC, U203 TPD4E1U06DBVR, U204 TPD4E1U06DBVR

Commit message: Dock v2 schematic fixes after review (J601 7-pin, Q602/R609, part data)
KiCad had the sheets open when the 7-pin pogo and the pull-up/veto parts were
added, and its save restored the old state. Restored now (KiCad closed):
- J601 -> Conn_01x07, footprint dock:Pogo-7; R606 4.7k (1.45 A)
- Q602 + R609 (POGO_OFF veto) added back to the pogo sheet
- L101 footprint L_TechFuse_SL0630 / LCSC C207841 again
- R406/R407 had the 1k LCSC number (copied from R405): now C25744; notes fixed
  on R406, R407, R504
- references back to the docs: C205->C107, R223->R106, R306->R201, R304->R202;
  R103/R104 swapped so R103 is on SCL and R104 on SDA (they were swapped, harmless)
- global label typo PD_SCA -> PD_SDA (both ends)
- net classes: 3V3_PWR, 5V_PWR (Power) and *USB_DP/*USB_DN/*USB_DM (USB),
  matching the labels used in the schematic

check_wiring.py: accepts interchangeable pins (R/C/button/crystal either way
round, TPD4E1U06 channels in any order), warns on a reversed L301/L401,
reports missing parts.

Co-Authored-By: Claude Opus 5.5 <noreply@anthropic.com>
Parts:
- renumbered R306 to R201, R304 to R202
Changed lines of the file:
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@@
 		(in_pos_files yes)
 		(dnp no)
-		(property "Reference" "R304"
+		(property "Reference" "R202"
 			(at 62.23 44.45 90)
 			(show_name no)
@@
 			(project "dock-v2"
 				(path "/928a9dc6-b0ce-4f47-a17d-f26fd77e396a/337fd23b-54e0-49b3-a4e7-e02473a7692d"
-					(reference "R304")
+					(reference "R202")
 					(unit 1)
 				)
@@
 		(in_pos_files yes)
 		(dnp no)
-		(property "Reference" "R306"
+		(property "Reference" "R201"
 			(at 57.912 33.274 90)
 			(show_name no)
@@
 			(project "dock-v2"
 				(path "/928a9dc6-b0ce-4f47-a17d-f26fd77e396a/337fd23b-54e0-49b3-a4e7-e02473a7692d"
-					(reference "R306")
+					(reference "R201")
 					(unit 1)
 				)
