File: hardware/dock-v2/ble.kicad_sch (KiCad schematic)
At the start: 11 parts, among them U501 ESP32-C3-MINI-1-H4X

Commit message: Dock v2 schematic fixes after review (J601 7-pin, Q602/R609, part data)
KiCad had the sheets open when the 7-pin pogo and the pull-up/veto parts were
added, and its save restored the old state. Restored now (KiCad closed):
- J601 -> Conn_01x07, footprint dock:Pogo-7; R606 4.7k (1.45 A)
- Q602 + R609 (POGO_OFF veto) added back to the pogo sheet
- L101 footprint L_TechFuse_SL0630 / LCSC C207841 again
- R406/R407 had the 1k LCSC number (copied from R405): now C25744; notes fixed
  on R406, R407, R504
- references back to the docs: C205->C107, R223->R106, R306->R201, R304->R202;
  R103/R104 swapped so R103 is on SCL and R104 on SDA (they were swapped, harmless)
- global label typo PD_SCA -> PD_SDA (both ends)
- net classes: 3V3_PWR, 5V_PWR (Power) and *USB_DP/*USB_DN/*USB_DM (USB),
  matching the labels used in the schematic

check_wiring.py: accepts interchangeable pins (R/C/button/crystal either way
round, TPD4E1U06 channels in any order), warns on a reversed L301/L401,
reports missing parts.

Co-Authored-By: Claude Opus 5.5 <noreply@anthropic.com>
Parts:
- R504: Note GPIO2 pull-up -> GPIO9 (BOOT) pull-up, beats A pull-down
Changed lines of the file:
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@@
 			)
 		)
-		(property "Note" "GPIO2 pull-up"
+		(property "Note" "GPIO9 (BOOT) pull-up, beats A pull-down"
 			(at 166.37 125.48 0)
 			(hide yes)
