File: hardware/dock-v2/mcu_b.kicad_sch (KiCad schematic)
At the start: 31 parts, among them SW401 SW_Push, U401 RP2354A, Y401 12MHz

Commit message: Dock v2 schematic fixes after review (J601 7-pin, Q602/R609, part data)
KiCad had the sheets open when the 7-pin pogo and the pull-up/veto parts were
added, and its save restored the old state. Restored now (KiCad closed):
- J601 -> Conn_01x07, footprint dock:Pogo-7; R606 4.7k (1.45 A)
- Q602 + R609 (POGO_OFF veto) added back to the pogo sheet
- L101 footprint L_TechFuse_SL0630 / LCSC C207841 again
- R406/R407 had the 1k LCSC number (copied from R405): now C25744; notes fixed
  on R406, R407, R504
- references back to the docs: C205->C107, R223->R106, R306->R201, R304->R202;
  R103/R104 swapped so R103 is on SCL and R104 on SDA (they were swapped, harmless)
- global label typo PD_SCA -> PD_SDA (both ends)
- net classes: 3V3_PWR, 5V_PWR (Power) and *USB_DP/*USB_DN/*USB_DM (USB),
  matching the labels used in the schematic

check_wiring.py: accepts interchangeable pins (R/C/button/crystal either way
round, TPD4E1U06 channels in any order), warns on a reversed L301/L401,
reports missing parts.

Co-Authored-By: Claude Opus 5.5 <noreply@anthropic.com>
Parts:
- R406: LCSC C11702 -> C25744; Note LED series -> B_RUN pull-up (beats A pull-down at reset)
- R407: LCSC C11702 -> C25744; Note LED series -> B_BOOTSEL pull-up (beats A pull-down)
Changed lines of the file:
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@@
 			)
 		)
-		(property "LCSC" "C11702"
+		(property "LCSC" "C25744"
 			(at 132.08 148.59 0)
 			(hide yes)
@@
 			)
 		)
-		(property "Note" "LED series"
+		(property "Note" "B_RUN pull-up (beats A pull-down at reset)"
 			(at 135.64 152.4 0)
 			(hide yes)
@@
 			)
 		)
-		(property "LCSC" "C11702"
+		(property "LCSC" "C25744"
 			(at 116.84 168.91 0)
 			(hide yes)
@@
 			)
 		)
-		(property "Note" "LED series"
+		(property "Note" "B_BOOTSEL pull-up (beats A pull-down)"
 			(at 120.4 172.72 0)
 			(hide yes)
