File: hardware/dock-v2/mcu_b.kicad_sch (KiCad schematic)
At the start: 31 parts, among them SW401 SW_Push, U401 RP2354A, Y401 12MHz

Commit message: Dock v2 schematic: pogo sheet wired, fixes from review (user's work, snapshot)
Connections:
- no-connect marks 26 -> 31
Changed lines of the file:
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@@
+	)
+	(no_connect
+		(at 132.08 172.72)
+	)
+	(no_connect
+		(at 132.08 180.34)
 	)
 	(no_connect
@@
 	)
 	(no_connect
+		(at 132.08 182.88)
+	)
+	(no_connect
 		(at 182.88 147.32)
 	)
@@
 	(no_connect
 		(at 182.88 205.74)
+	)
+	(no_connect
+		(at 132.08 175.26)
 	)
 	(no_connect
@@
 	)
 	(no_connect
+		(at 132.08 177.8)
+	)
+	(no_connect
