File: hardware/dock-v2/mcu_b.kicad_sch (KiCad schematic)
At the start: 31 parts, among them SW401 SW_Push, U401 RP2354A, Y401 12MHz

Commit message: Dock v2: routing complete, SWD test pads removed (user's work, snapshot)
Co-Authored-By: Claude Opus 5.5 <noreply@anthropic.com>
Parts:
- removed TP401, TP402, TP403: TestPoint, TestPoint:TestPoint_Pad_D1.0mm, symbol Connector:TestPoint

Commit message: Dock v2 PCB: fix unconnected nets, widen power traces, readable silkscreen, 2 copper layers
- MCU A and B IOVDD (pins 30/38) had no 3V3 feed: added an under-chip jumper (A)
  and a top-layer feed to the 3V3 via by the buck (B)
- MCU B's exposed pad sat in a GND pour island: 3V3 bottom ring via moved so the
  plane reaches it; crystal B GND vias added; pour clearance 0.5 -> 0.3 mm
- power traces widened where clearance allows (switch node 1.5 mm, 5 V 1.0 mm,
  VBUS_IN/POGO_5V/KBD_VBUS as far as fits); VBUS_IN vias 0.8/0.4
- silkscreen: refs 0.8/1.0 mm, re-placed clear of pads and parts, labels for
  connectors, buttons, LEDs and ESP32 UART pads; 22 small passives hidden
- copper layers 4 -> 2 (inner layers were empty)
- model/docs: SWD test pads TP301-303/TP401-403 removed

DRC: 0 violations, 0 unconnected, 0 parity issues.

Co-Authored-By: Claude Opus 5.5 <noreply@anthropic.com>
Parts:
- added J501: Conn_01x03, Connector_PinHeader_2.54mm:PinHeader_1x03_P2.54mm_Vertical, symbol Connector_Generic:Conn_01x03
Connections:
- net B_SWCLK: now also J501.3 (Pin_3)
- net B_SWDIO: now also J501.2 (Pin_2)
- net GND: now also J501.1 (Pin_1)
Changed lines of the file:
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@@
+	)
+	(junction
+		(at 113.03 210.82)
+		(diameter 0)
+		(color 0 0 0 0)
 	)
 	(junction
@@
 	)
 	(junction
+		(at 111.76 208.28)
+		(diameter 0)
+		(color 0 0 0 0)
+	)
+	(junction
 		(at 165.1 129.54)
 		(diameter 0)
@@
 	(wire
 		(pts
-			(xy 93.98 208.28) (xy 132.08 208.28)
+			(xy 93.98 208.28) (xy 111.76 208.28)
 		)
 		(stroke
@@
 	(wire
 		(pts
+			(xy 107.95 218.44) (xy 111.76 218.44)
+		)
+		(stroke
+			(width 0)
+			(type default)
+		)
+	)
+	(wire
+		(pts
 			(xy 118.11 97.79) (xy 124.46 97.79)
 		)
@@
 	(wire
 		(pts
-			(xy 93.98 210.82) (xy 132.08 210.82)
+			(xy 111.76 208.28) (xy 132.08 208.28)
+		)
+		(stroke
+			(width 0)
+			(type default)
+		)
+	)
+	(wire
+		(pts
+			(xy 111.76 208.28) (xy 111.76 218.44)
+		)
+		(stroke
+			(width 0)
+			(type default)
+		)
+	)
+	(wire
+		(pts
+			(xy 93.98 210.82) (xy 113.03 210.82)
 		)
 		(stroke
@@
 	(wire
 		(pts
+			(xy 107.95 220.98) (xy 113.03 220.98)
+		)
+		(stroke
+			(width 0)
+			(type default)
+		)
+	)
+	(wire
+		(pts
 			(xy 144.78 105.41) (xy 144.78 97.79)
 		)
@@
 	(wire
 		(pts
+			(xy 113.03 220.98) (xy 113.03 210.82)
+		)
+		(stroke
+			(width 0)
+			(type default)
+		)
+	)
+	(wire
+		(pts
 			(xy 137.16 105.41) (xy 144.78 105.41)
+		)
+		(stroke
+			(width 0)
+			(type default)
+		)
+	)
+	(wire
+		(pts
+			(xy 113.03 210.82) (xy 132.08 210.82)
 		)
 		(stroke
@@
 				(path "/928a9dc6-b0ce-4f47-a17d-f26fd77e396a/da035690-56be-4ab0-b555-b768c130331c"
 					(reference "R406")
+					(unit 1)
+				)
+			)
+		)
+	)
+	(symbol
+		(lib_id "Connector_Generic:Conn_01x03")
+		(at 102.87 220.98 180)
+		(unit 1)
+		(body_style 1)
+		(exclude_from_sim no)
+		(in_bom yes)
+		(on_board yes)
+		(in_pos_files yes)
+		(dnp no)
+		(fields_autoplaced yes)
+		(property "Reference" "J501"
+			(at 102.87 212.09 0)
+			(show_name no)
+			(do_not_autoplace no)
+			(effects
+				(font
+					(size 1.27 1.27)
+				)
+			)
+		)
+		(property "Value" "Conn_01x03"
+			(at 102.87 214.63 0)
+			(show_name no)
+			(do_not_autoplace no)
+			(effects
+				(font
+					(size 1.27 1.27)
+				)
+			)
+		)
+		(property "Footprint" "Connector_PinHeader_2.54mm:PinHeader_1x03_P2.54mm_Vertical"
+			(at 102.87 220.98 0)
+			(hide yes)
+			(show_name no)
+			(do_not_autoplace no)
+			(effects
+				(font
+					(size 1.27 1.27)
+				)
+			)
+		)
+		(property "Datasheet" ""
+			(at 102.87 220.98 0)
+			(hide yes)
+			(show_name no)
+			(do_not_autoplace no)
+			(effects
+				(font
+					(size 1.27 1.27)
+				)
+			)
+		)
+		(property "Description" "Generic connector, single row, 01x03, script generated (kicad-library-utils/schlib/autogen/connector/)"
+			(at 102.87 220.98 0)
+			(hide yes)
+			(show_name no)
+			(do_not_autoplace no)
+			(effects
+				(font
+					(size 1.27 1.27)
+				)
+			)
+		)
+		(pin "3"
+		)
+		(pin "1"
+		)
+		(pin "2"
+		)
+		(instances
+			(project "dock-v2"
+				(path "/928a9dc6-b0ce-4f47-a17d-f26fd77e396a/da035690-56be-4ab0-b555-b768c130331c"
+					(reference "J501")
 					(unit 1)
 				)
@@
 					(unit 1)
 				)
+			)
+		)
+	)
+	(symbol
+		(lib_id "power:GND")
+		(at 107.95 223.52 90)
+		(unit 1)
+		(body_style 1)
+		(exclude_from_sim no)
+		(in_bom yes)
+		(on_board yes)
+		(in_pos_files yes)
+		(dnp no)
+		(fields_autoplaced yes)
+		(property "Reference" "#PWR0511"
+			(at 114.3 223.52 0)
+			(hide yes)
+			(show_name no)
+			(do_not_autoplace no)
+			(effects
+				(font
+					(size 1.27 1.27)
+				)
+			)
+		)
+		(property "Value" "GND"
+			(at 111.76 223.5199 90)
+			(show_name no)
+			(do_not_autoplace no)
+			(effects
+				(font
+					(size 1.27 1.27)
+				)
+				(justify right)
+			)
+		)
+		(property "Footprint" ""
+			(at 107.95 223.52 0)
+			(hide yes)
+			(show_name no)
+			(do_not_autoplace no)
+			(effects
+				(font
+					(size 1.27 1.27)
+				)
+			)
+		)
+		(property "Datasheet" ""
+			(at 107.95 223.52 0)
+			(hide yes)
+			(show_name no)
+			(do_not_autoplace no)
+			(effects
+				(font
+					(size 1.27 1.27)
+				)
+			)
+		)
+		(property "Description" "Power symbol creates a global label with name \"GND\" , ground"
+			(at 107.95 223.52 0)
+			(hide yes)
+			(show_name no)
+			(do_not_autoplace no)
+			(effects
+				(font
+					(size 1.27 1.27)
+				)
+			)
+		)
+		(pin "1"
+		)
+		(instances
+			(project "dock-v2"
+				(path "/928a9dc6-b0ce-4f47-a17d-f26fd77e396a/da035690-56be-4ab0-b555-b768c130331c"
+					(reference "#PWR0511")
+					(unit 1)
+				)
