File: hardware/dock-v2/power.kicad_sch (KiCad schematic)
At the start: 27 parts, among them J101 TYPE-C-31-M-12, U101 TPD4E1U06DBVR, U102 CH224A, U103 TPS54331DR, U104 AMS1117-3.3

Commit message: Dock v2 schematic fixes after review (J601 7-pin, Q602/R609, part data)
KiCad had the sheets open when the 7-pin pogo and the pull-up/veto parts were
added, and its save restored the old state. Restored now (KiCad closed):
- J601 -> Conn_01x07, footprint dock:Pogo-7; R606 4.7k (1.45 A)
- Q602 + R609 (POGO_OFF veto) added back to the pogo sheet
- L101 footprint L_TechFuse_SL0630 / LCSC C207841 again
- R406/R407 had the 1k LCSC number (copied from R405): now C25744; notes fixed
  on R406, R407, R504
- references back to the docs: C205->C107, R223->R106, R306->R201, R304->R202;
  R103/R104 swapped so R103 is on SCL and R104 on SDA (they were swapped, harmless)
- global label typo PD_SCA -> PD_SDA (both ends)
- net classes: 3V3_PWR, 5V_PWR (Power) and *USB_DP/*USB_DN/*USB_DM (USB),
  matching the labels used in the schematic

check_wiring.py: accepts interchangeable pins (R/C/button/crystal either way
round, TPD4E1U06 channels in any order), warns on a reversed L301/L401,
reports missing parts.

Co-Authored-By: Claude Opus 5.5 <noreply@anthropic.com>
Parts:
- L101: footprint (none) -> Inductor_SMD:L_TechFuse_SL0630; LCSC C10167 -> C207841; Note SMDRH105R-6R8NT (Ext) or a Basic 6.8 uH, 3 A+: pick footpri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 -> SLO0630H6R8MTT: Isat 8 A (> 5.8 A max current limit), 45 mO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
- R103: renamed from R104; Note SDA pull-up to 3V3 -> SCL pull-up to 3V3
- R104: renamed from R103; Note SCL pull-up to 3V3 -> SDA pull-up to 3V3
- renumbered C205 to C107, R223 to R106
Connections:
- net PD_SCA renamed PD_SDA
Changed lines of the file:
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@@
 		)
 	)
-	(global_label "PD_SCA"
+	(global_label "PD_SDA"
 		(shape input)
 		(at 104.14 48.26 270)
@@
 		(in_pos_files yes)
 		(dnp no)
-		(property "Reference" "R103"
+		(property "Reference" "R104"
 			(at 120.65 50.292 90)
 			(show_name no)
@@
 			)
 		)
-		(property "Note" "SCL pull-up to 3V3"
+		(property "Note" "SDA pull-up to 3V3"
 			(at 121.92 44.7 0)
 			(hide yes)
@@
 			(project "dock-v2"
 				(path "/928a9dc6-b0ce-4f47-a17d-f26fd77e396a/211f96f8-19fe-45b9-be96-b177c1b5d6c4"
-					(reference "R103")
+					(reference "R104")
 					(unit 1)
 				)
@@
 		(in_pos_files yes)
 		(dnp no)
-		(property "Reference" "C205"
+		(property "Reference" "C107"
 			(at 186.182 46.228 0)
 			(show_name no)
@@
 			(project "dock-v2"
 				(path "/928a9dc6-b0ce-4f47-a17d-f26fd77e396a/211f96f8-19fe-45b9-be96-b177c1b5d6c4"
-					(reference "C205")
+					(reference "C107")
 					(unit 1)
 				)
@@
 		(in_pos_files yes)
 		(dnp no)
-		(property "Reference" "R104"
+		(property "Reference" "R103"
 			(at 120.396 45.466 90)
 			(show_name no)
@@
 			)
 		)
-		(property "Note" "SDA pull-up to 3V3"
+		(property "Note" "SCL pull-up to 3V3"
 			(at 121.92 39.62 0)
 			(hide yes)
@@
 			(project "dock-v2"
 				(path "/928a9dc6-b0ce-4f47-a17d-f26fd77e396a/211f96f8-19fe-45b9-be96-b177c1b5d6c4"
-					(reference "R104")
+					(reference "R103")
 					(unit 1)
 				)
@@
 		(in_pos_files yes)
 		(dnp no)
-		(property "Reference" "R223"
+		(property "Reference" "R106"
 			(at 211.836 44.196 90)
 			(show_name no)
@@
 			(project "dock-v2"
 				(path "/928a9dc6-b0ce-4f47-a17d-f26fd77e396a/211f96f8-19fe-45b9-be96-b177c1b5d6c4"
-					(reference "R223")
+					(reference "R106")
 					(unit 1)
 				)
@@
 			)
 		)
-		(property "Footprint" ""
+		(property "Footprint" "Inductor_SMD:L_TechFuse_SL0630"
 			(at 215.9 41.91 0)
 			(hide yes)
@@
 			)
 		)
-		(property "LCSC" "C10167"
+		(property "LCSC" "C207841"
 			(at 215.9 41.91 0)
 			(hide yes)
@@
 			)
 		)
-		(property "Note" "SMDRH105R-6R8NT (Ext) or a Basic 6.8 uH, 3 A+: pick footprint"
+		(property "Note" "SLO0630H6R8MTT: Isat 8 A (> 5.8 A max current limit), 45 mOhm, 7.1x6.6x3.0"
 			(at 219.07 45.72 0)
 			(hide yes)
