File: hardware/dock-v2/dock-v2.kicad_pcb (KiCad board)
At the start: 4 copper layers, 0 parts

Commit message: Dock v2: PCB placement in progress (user's work, snapshot)
Parts:
- added C101: 1uF, Capacitor_SMD:C_0603_1608Metric, F.Cu at (227.5, 71.0)
- added C102: 10uF, Capacitor_SMD:C_0805_2012Metric, F.Cu at (212.0, 73.0)
- added C103: 10uF, Capacitor_SMD:C_0805_2012Metric, F.Cu at (212.0, 76.5)
- added C104: 100nF, Capacitor_SMD:C_0402_1005Metric, F.Cu at (207.0, 66.5)
- added C105: 10nF, Capacitor_SMD:C_0402_1005Metric, F.Cu at (215.5, 70.0)
- added C106: 4.7nF, Capacitor_SMD:C_0402_1005Metric, F.Cu at (209.5, 61.5)
- added C107: 47pF, Capacitor_SMD:C_0402_1005Metric, F.Cu at (211.0, 61.5)
- added C108: 22uF 25V, Capacitor_SMD:C_1206_3216Metric, F.Cu at (193.5, 76.5)
- added C109: 22uF 25V, Capacitor_SMD:C_1206_3216Metric, F.Cu at (193.5, 72.0)
- added C110: 22uF 25V, Capacitor_SMD:C_1206_3216Metric, F.Cu at (193.5, 69.0)
- added C111: 10uF, Capacitor_SMD:C_0805_2012Metric, F.Cu at (199.5, 54.0)
- added C112: 10uF, Capacitor_SMD:C_0805_2012Metric, F.Cu at (206.0, 54.0)
- added C201: 220uF 16V, dock_v2:CP_Radial_D6.3mm_P5.00mm, F.Cu at (130.5, 77.0)
- added C202: 10uF, Capacitor_SMD:C_0805_2012Metric, F.Cu at (132.6, 74.0)
- added C203: 1uF, Capacitor_SMD:C_0402_1005Metric, F.Cu at (134.1, 74.0)
- added C204: 1uF, Capacitor_SMD:C_0402_1005Metric, F.Cu at (138.1, 76.5)
- added C301: 4.7uF, dock_v2:C_0402_RPi_Wide, F.Cu at (167.0, 23.5)
- added C302: 4.7uF, dock_v2:C_0402_RPi_Wide, F.Cu at (166.5, 20.0)
- added C303: 4.7uF, Capacitor_SMD:C_0402_1005Metric, F.Cu at (169.0, 24.0)
- added C304: 100nF, Capacitor_SMD:C_0402_1005Metric, F.Cu at (166.5, 19.0)
- added C305: 100nF, Capacitor_SMD:C_0402_1005Metric, F.Cu at (168.5, 19.0)
- added C306: 100nF, Capacitor_SMD:C_0402_1005Metric, F.Cu at (168.5, 20.0)
- added C307: 100nF, Capacitor_SMD:C_0402_1005Metric, F.Cu at (172.5, 23.0)
- added C308: 100nF, Capacitor_SMD:C_0402_1005Metric, F.Cu at (172.5, 22.0)
- added C309: 100nF, Capacitor_SMD:C_0402_1005Metric, F.Cu at (175.0, 26.0)
- added C310: 100nF, Capacitor_SMD:C_0402_1005Metric, F.Cu at (178.9, 34.0)
- added C311: 100nF, Capacitor_SMD:C_0402_1005Metric, F.Cu at (178.9, 35.9)
- added C312: 100nF, Capacitor_SMD:C_0402_1005Metric, F.Cu at (178.9, 37.9)
- added C313: 100nF, Capacitor_SMD:C_0402_1005Metric, F.Cu at (185.5, 30.5)
- added C314: 10uF, Capacitor_SMD:C_0805_2012Metric, F.Cu at (184.0, 40.0)
- added C315: 15pF, Capacitor_SMD:C_0402_1005Metric, F.Cu at (164.5, 35.0)
- added C316: 15pF, Capacitor_SMD:C_0402_1005Metric, F.Cu at (161.2, 37.4)
- added C401: 4.7uF, dock_v2:C_0402_RPi_Wide, F.Cu at (189.6, 148.7)
- added C402: 4.7uF, dock_v2:C_0402_RPi_Wide, F.Cu at (189.6, 150.3)
- added C403: 4.7uF, Capacitor_SMD:C_0402_1005Metric, F.Cu at (192.7, 135.0)
- added C404: 100nF, Capacitor_SMD:C_0402_1005Metric, F.Cu at (192.7, 137.0)
- added C405: 100nF, Capacitor_SMD:C_0402_1005Metric, F.Cu at (192.7, 138.9)
- added C406: 100nF, Capacitor_SMD:C_0402_1005Metric, F.Cu at (192.7, 140.9)
- added C407: 100nF, Capacitor_SMD:C_0402_1005Metric, F.Cu at (192.7, 142.9)
- added C408: 100nF, Capacitor_SMD:C_0402_1005Metric, F.Cu at (195.5, 135.0)
- added C409: 100nF, Capacitor_SMD:C_0402_1005Metric, F.Cu at (195.5, 137.0)
- added C410: 100nF, Capacitor_SMD:C_0402_1005Metric, F.Cu at (195.5, 138.9)
- added C411: 100nF, Capacitor_SMD:C_0402_1005Metric, F.Cu at (195.5, 140.9)
- added C412: 100nF, Capacitor_SMD:C_0402_1005Metric, F.Cu at (195.5, 142.9)
- added C413: 100nF, Capacitor_SMD:C_0402_1005Metric, F.Cu at (198.4, 135.0)
- added C414: 10uF, Capacitor_SMD:C_0805_2012Metric, F.Cu at (208.0, 135.0)
- added C415: 15pF, Capacitor_SMD:C_0402_1005Metric, F.Cu at (176.5, 63.0)
- added C416: 15pF, Capacitor_SMD:C_0402_1005Metric, F.Cu at (179.5, 60.5)
- added C501: 1uF, Capacitor_SMD:C_0402_1005Metric, F.Cu at (215.5, 106.0)
- added C502: 10uF, Capacitor_SMD:C_0805_2012Metric, F.Cu at (221.5, 104.5)
- added C503: 100nF, Capacitor_SMD:C_0402_1005Metric, F.Cu at (222.5, 106.0)
- added C601: 1uF, Capacitor_SMD:C_0402_1005Metric, F.Cu at (186.0, 123.8)
- added C602: 10uF, Capacitor_SMD:C_0805_2012Metric, F.Cu at (178.1, 130.2)
- added C603: 1uF, Capacitor_SMD:C_0402_1005Metric, F.Cu at (186.0, 125.7)
- added D101: SMBJ15A, Diode_SMD:D_SMB, F.Cu at (230.5, 56.5)
- added D102: SS54, Diode_SMD:D_SMC, F.Cu at (199.5, 73.0)
- added D301: LED red, LED_SMD:LED_0603_1608Metric, F.Cu at (156.2, 27.4)
- added D401: LED red, LED_SMD:LED_0603_1608Metric, F.Cu at (170.5, 51.0)
- added J101: TYPE-C-31-M-12, Connector_USB:USB_C_Receptacle_HRO_TYPE-C-31-M-12, F.Cu at (234.0, 65.0)
- added J201: TYPE-C-31-M-12, Connector_USB:USB_C_Receptacle_HRO_TYPE-C-31-M-12, F.Cu at (125.0, 64.5)
- added J202: TYPE-C-31-M-12, Connector_USB:USB_C_Receptacle_HRO_TYPE-C-31-M-12, F.Cu at (126.2, 34.5)
- added J203: TYPE-C-31-M-12, Connector_USB:USB_C_Receptacle_HRO_TYPE-C-31-M-12, F.Cu at (233.2, 35.0)
- added J601: Pogo 7-pin, dock:Pogo-7, F.Cu at (180.2, 119.9)
- added L101: 6.8uH, Inductor_SMD:L_TechFuse_SL0630, F.Cu at (199.5, 62.5)
- added L301: 3.3uH, dock_v2:L_Abracon_AOTA-B201610S3R3_0806, F.Cu at (166.5, 21.5)
- added L401: 3.3uH, dock_v2:L_Abracon_AOTA-B201610S3R3_0806, F.Cu at (206.0, 151.9)
- added Q601: 2N7002, Package_TO_SOT_SMD:SOT-23, F.Cu at (173.4, 125.0)
- added Q602: 2N7002, Package_TO_SOT_SMD:SOT-23, F.Cu at (173.4, 129.4)
- added R101: 6.8k, Resistor_SMD:R_0402_1005Metric, F.Cu at (220.5, 72.5)
- added R102: 10k, Resistor_SMD:R_0402_1005Metric, F.Cu at (221.5, 72.5)
- added R103: 4.7k, Resistor_SMD:R_0402_1005Metric, F.Cu at (221.0, 61.0)
- added R104: 4.7k, Resistor_SMD:R_0402_1005Metric, F.Cu at (220.0, 59.5)
- added R105: 51k, Resistor_SMD:R_0402_1005Metric, F.Cu at (210.5, 59.5)
- added R106: 12k, Resistor_SMD:R_0402_1005Metric, F.Cu at (206.5, 62.5)
- added R107: 2.2k, Resistor_SMD:R_0402_1005Metric, F.Cu at (213.5, 60.5)
- added R201: 33k, Resistor_SMD:R_0402_1005Metric, F.Cu at (135.0, 61.0)
- added R202: 33k, Resistor_SMD:R_0402_1005Metric, F.Cu at (135.0, 68.5)
- added R203: 15k, Resistor_SMD:R_0402_1005Metric, F.Cu at (136.5, 66.0)
- added R204: 15k, Resistor_SMD:R_0402_1005Metric, F.Cu at (136.5, 63.5)
- added R205: 22, Resistor_SMD:R_0402_1005Metric, F.Cu at (139.5, 65.5)
- added R206: 22, Resistor_SMD:R_0402_1005Metric, F.Cu at (139.5, 64.0)
- added R207: 6.8k, Resistor_SMD:R_0402_1005Metric, F.Cu at (134.5, 80.5)
- added R208: 100k, Resistor_SMD:R_0402_1005Metric, F.Cu at (138.1, 78.5)
- added R209: 10k, Resistor_SMD:R_0402_1005Metric, F.Cu at (136.0, 73.0)
- added R210: 15k, Resistor_SMD:R_0402_1005Metric, F.Cu at (138.0, 73.5)
- added R211: 5.1k, Resistor_SMD:R_0402_1005Metric, F.Cu at (130.5, 43.5)
- added R212: 5.1k, Resistor_SMD:R_0402_1005Metric, F.Cu at (121.5, 43.0)
- added R213: 22k, Resistor_SMD:R_0402_1005Metric, F.Cu at (130.0, 40.5)
- added R214: 33k, Resistor_SMD:R_0402_1005Metric, F.Cu at (132.0, 40.0)
- added R215: 22, Resistor_SMD:R_0402_1005Metric, F.Cu at (124.5, 45.5)
- added R216: 22, Resistor_SMD:R_0402_1005Metric, F.Cu at (128.0, 45.5)
- added R217: 5.1k, Resistor_SMD:R_0402_1005Metric, F.Cu at (237.0, 41.5)
- added R218: 5.1k, Resistor_SMD:R_0402_1005Metric, F.Cu at (228.0, 44.0)
- added R219: 22k, Resistor_SMD:R_0402_1005Metric, F.Cu at (228.5, 41.0)
- added R220: 33k, Resistor_SMD:R_0402_1005Metric, F.Cu at (226.5, 40.0)
- added R221: 22, Resistor_SMD:R_0402_1005Metric, F.Cu at (231.5, 46.0)
- added R222: 22, Resistor_SMD:R_0402_1005Metric, F.Cu at (234.5, 46.0)
- added R301: 33, Resistor_SMD:R_0402_1005Metric, F.Cu at (170.5, 25.5)
- added R302: 1k, Resistor_SMD:R_0402_1005Metric, F.Cu at (165.0, 40.0)
- added R303: 1k, Resistor_SMD:R_0402_1005Metric, F.Cu at (159.5, 25.0)
- added R305: 1k, Resistor_SMD:R_0402_1005Metric, F.Cu at (159.2, 27.4)
- added R401: 33, Resistor_SMD:R_0402_1005Metric, F.Cu at (189.8, 135.0)
- added R402: 1k, Resistor_SMD:R_0402_1005Metric, F.Cu at (182.0, 60.5)
- added R403: 1k, Resistor_SMD:R_0402_1005Metric, F.Cu at (189.8, 139.0)
- added R404: 1k, Resistor_SMD:R_0402_1005Metric, F.Cu at (189.8, 141.0)
- added R405: 1k, Resistor_SMD:R_0402_1005Metric, F.Cu at (173.0, 51.0)
- added R406: 10k, Resistor_SMD:R_0402_1005Metric, F.Cu at (189.8, 145.0)
- added R407: 10k, Resistor_SMD:R_0402_1005Metric, F.Cu at (189.8, 147.0)
- added R501: 10k, Resistor_SMD:R_0402_1005Metric, F.Cu at (216.5, 105.0)
- added R502: 10k, Resistor_SMD:R_0402_1005Metric, F.Cu at (210.0, 116.5)
- added R503: 10k, Resistor_SMD:R_0402_1005Metric, F.Cu at (218.5, 105.0)
- added R504: 10k, Resistor_SMD:R_0402_1005Metric, F.Cu at (210.0, 117.5)
- added R601: 1k, Resistor_SMD:R_0402_1005Metric, F.Cu at (177.3, 123.8)
- added R602: 1k, Resistor_SMD:R_0402_1005Metric, F.Cu at (177.3, 125.8)
- added R603: 1k, Resistor_SMD:R_0402_1005Metric, F.Cu at (177.3, 127.7)
- added R604: 10k, Resistor_SMD:R_0402_1005Metric, F.Cu at (180.2, 123.8)
- added R605: 100k, Resistor_SMD:R_0402_1005Metric, F.Cu at (180.2, 125.8)
- added R606: 4.7k, Resistor_SMD:R_0402_1005Metric, F.Cu at (180.2, 127.7)
- added R607: 10k, Resistor_SMD:R_0402_1005Metric, F.Cu at (183.2, 123.8)
- added R608: 15k, Resistor_SMD:R_0402_1005Metric, F.Cu at (183.2, 125.8)
- added R609: 100k, Resistor_SMD:R_0402_1005Metric, F.Cu at (183.2, 127.7)
- added SW301: SW_Push, Button_Switch_SMD:SW_Push_1P1T_XKB_TS-1187A, F.Cu at (150.5, 26.0)
- added SW302: SW_Push, Button_Switch_SMD:SW_Push_1P1T_XKB_TS-1187A, F.Cu at (143.3, 128.9)
- added SW401: SW_Push, Button_Switch_SMD:SW_Push_1P1T_XKB_TS-1187A, F.Cu at (204.2, 147.2)
- added TP301: TestPoint, TestPoint:TestPoint_Pad_D1.0mm, F.Cu at (157.7, 120.4)
- added TP302: TestPoint, TestPoint:TestPoint_Pad_D1.0mm, F.Cu at (157.7, 123.5)
- added TP303: TestPoint, TestPoint:TestPoint_Pad_D1.0mm, F.Cu at (157.7, 126.5)
- added TP401: TestPoint, TestPoint:TestPoint_Pad_D1.0mm, F.Cu at (201.4, 135.5)
- added TP402: TestPoint, TestPoint:TestPoint_Pad_D1.0mm, F.Cu at (201.4, 138.6)
- added TP403: TestPoint, TestPoint:TestPoint_Pad_D1.0mm, F.Cu at (201.4, 141.6)
- added TP503: TestPoint, TestPoint:TestPoint_Pad_D1.0mm, F.Cu at (219.0, 122.0)
- added TP504: TestPoint, TestPoint:TestPoint_Pad_D1.0mm, F.Cu at (216.5, 122.0)
- added TP505: TestPoint, TestPoint:TestPoint_Pad_D1.0mm, F.Cu at (214.0, 122.0)
- added U101: TPD4E1U06DBVR, Package_TO_SOT_SMD:SOT-23-6, F.Cu at (225.5, 65.5)
- added U102: CH224A, Package_SO:SSOP-10-1EP_3.9x4.9mm_P1mm_EP2.1x3.3mm, F.Cu at (219.5, 66.0)
- added U103: TPS54331DR, Package_SO:SOIC-8_3.9x4.9mm_P1.27mm, F.Cu at (211.5, 66.5)
- added U104: AMS1117-3.3, Package_TO_SOT_SMD:SOT-223-3_TabPin2, F.Cu at (212.5, 55.0)
- added U201: TPD4E1U06DBVR, Package_TO_SOT_SMD:SOT-23-6, F.Cu at (134.0, 64.5)
- added U202: SY6280AAC, Package_TO_SOT_SMD:SOT-23-5, F.Cu at (135.1, 78.0)
- added U203: TPD4E1U06DBVR, Package_TO_SOT_SMD:SOT-23-6, F.Cu at (126.0, 43.0)
- added U204: TPD4E1U06DBVR, Package_TO_SOT_SMD:SOT-23-6, F.Cu at (233.0, 43.0)
- added U301: RP2354A, dock_v2:RP2350A_QFN-60_RPi_Vias, F.Cu at (165.7, 29.0)
- added U401: RP2354A, dock_v2:RP2350A_QFN-60_RPi_Vias, F.Cu at (179.5, 52.0)
- added U501: ESP32-C3-MINI-1-H4X, dock_v2:ESP32-C3-MINI-1, F.Cu at (220.8, 113.3)
- added U601: TPD4E1U06DBVR, Package_TO_SOT_SMD:SOT-23-6, F.Cu at (168.4, 125.2)
- added U602: SY6280AAC, Package_TO_SOT_SMD:SOT-23-5, F.Cu at (168.4, 129.8)
- added Y301: 12MHz, Crystal:Crystal_SMD_3225-4Pin_3.2x2.5mm, F.Cu at (164.0, 37.5)
- added Y401: 12MHz, Crystal:Crystal_SMD_3225-4Pin_3.2x2.5mm, F.Cu at (179.5, 63.0)
Routing:
- net GND: track 0.00 -> 200.4 mm, vias 0 -> 11
- net 3V3_PWR: track 0.00 -> 106.9 mm, vias 0 -> 7
- net /POWER/VBUS_IN: track 0.00 -> 53.5 mm, vias 0 -> 4
- net KBD_VBUS_EN: track 0.00 -> 46.9 mm
- net 5V_PWR: track 0.00 -> 41.2 mm
- net KBD_VBUS: track 0.00 -> 29.2 mm, vias 0 -> 2
- net /MCU_A/A_1V1: track 0.00 -> 25.0 mm, vias 0 -> 3
- net PRS_USB_DN: track 0.00 -> 17.6 mm
- net POWER_USB_DM: track 0.00 -> 17.5 mm, vias 0 -> 2
- net Net-(J101-CC2): track 0.00 -> 17.3 mm
- net Net-(D102-K): track 0.00 -> 16.7 mm
- net Net-(U201-D2-): track 0.00 -> 14.3 mm
- net Net-(J101-CC1): track 0.00 -> 14.1 mm
- net POWER_USB_DN: track 0.00 -> 13.9 mm, vias 0 -> 2
- net Net-(U103-VSENSE): track 0.00 -> 13.8 mm, vias 0 -> 2
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- added copper zone on F.Cu, net GND
