File: hardware/dock-v2/dock-v2.kicad_pcb (KiCad board)
At the start: 4 copper layers, 100 x 100 mm, 148 parts, among them J101 TYPE-C-31-M-12, J201 TYPE-C-31-M-12, J202 TYPE-C-31-M-12, J203 TYPE-C-31-M-12, J601 Pogo 7-pin, Q601 2N7002, Q602 2N7002, SW301 SW_Push, SW302 SW_Push, SW401 SW_Push, U101 TPD4E1U06DBVR, U102 CH224A, U103 TPS54331DR, U104 AMS1117-3.3, U201 TPD4E1U06DBVR, U202 SY6280AAC, U203 TPD4E1U06DBVR, U204 TPD4E1U06DBVR, U301 RP2354A, U401 RP2354A, U501 ESP32-C3-MINI-1-H4X, U601 TPD4E1U06DBVR, U602 SY6280AAC, Y301 12MHz, Y401 12MHz

Commit message: Dock v2: placement and partial routing (user's work, snapshot)
Parts:
- moved TP403 96.4 mm to (203.2, 45.2)
- moved TP401 96.4 mm to (203.2, 39.1)
- moved TP402 96.4 mm to (203.2, 42.2)
- moved SW401 88.0 mm to (169.0, 66.5)
- moved L401 84.8 mm to (177.5, 72.0)
- moved C402 81.2 mm to (177.5, 70.0), turned to 180 degrees
- moved C412 79.5 mm to (179.5, 65.0), turned to 180 degrees
- moved C414 77.7 mm to (177.5, 63.5), turned to -90 degrees
- moved C411 77.1 mm to (177.5, 66.0)
- moved R407 75.5 mm to (170.5, 74.0), turned to 180 degrees
- moved C401 75.2 mm to (181.0, 74.0), turned to -90 degrees
- moved C407 75.1 mm to (179.5, 69.0)
- moved C410 74.7 mm to (179.5, 66.0)
- moved C406 73.5 mm to (177.5, 69.0)
- moved C413 73.5 mm to (179.5, 64.0), turned to 180 degrees
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Connections:
- U601 pad 3: Net-(J601-Pin_4) -> Net-(J601-Pin_3)
- U601 pad 4: Net-(J601-Pin_3) -> Net-(J601-Pin_4)
Routing:
- net GND: track 200.4 -> 361.8 mm, vias 11 -> 14
- net 3V3_PWR: track 106.9 -> 161.4 mm, vias 7 -> 6
- net KBD_VBUS_EN: track 46.9 -> 1.91 mm
- net POGO_5V: track 0.00 -> 30.8 mm, vias 0 -> 1
- net POGO_DET: track 0.00 -> 18.8 mm
- net PRS_USB_DN: track 17.6 -> 0.00 mm
- net Net-(Q601-D): track 0.00 -> 14.5 mm
- net /MCU_A/A_1V1: track 25.0 -> 12.8 mm, vias 3 -> 0
- net PRS_USB_DP: track 11.9 -> 0.00 mm
- net /MCU_B/B_1V1: track 0.00 -> 11.6 mm
- net /POWER/VBUS_IN: track 53.5 -> 42.1 mm
- net 5V_PWR: track 41.2 -> 30.1 mm, vias 0 -> 1
- net Net-(R403-Pad1): track 0.00 -> 9.62 mm
- net Net-(J601-Pin_3): track 0.00 -> 9.21 mm
- net Net-(J601-Pin_4): track 0.00 -> 8.27 mm
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- added copper zone on B.Cu, net GND
- removed copper zone on F.Cu, net GND
