File: hardware/dock-v2/dock-v2.kicad_pcb (KiCad board)
At the start: 2 copper layers, 100 x 100 mm, 154 parts, among them J101 TYPE-C-31-M-12, J201 TYPE-C-31-M-12, J202 TYPE-C-31-M-12, J203 TYPE-C-31-M-12, J401 Conn_01x03, J501 Conn_01x03, J601 B7B-XH-A (to lid pogo board), Q601 2N7002, Q602 2N7002, SW301 SW_Push, SW302 SW_Push, SW401 SW_Push, U101 TPD4E1U06DBVR, U102 CH224A, U103 TPS54331DR, U104 AMS1117-3.3, U201 TPD4E1U06DBVR, U202 SY6280AAC, U203 TPD4E1U06DBVR, U204 TPD4E1U06DBVR, U301 RP2354A, U401 RP2354A, U501 ESP32-C3-MINI-1-H4X, U601 TPD4E1U06DBVR, U602 SY6280AAC, Y301 12MHz, Y401 12MHz

Commit message: Pad v2 decisions: ESP32-S3-MINI-1-N8, docks on top, 1x 21700-50E + ETA6003 (research docs)
Co-Authored-By: Claude Opus 5.5 <noreply@anthropic.com>
Parts:
- moved H10 96.9 mm to (133.0, 58.0)
- moved H3 79.3 mm to (210.0, 39.0)
- moved H5 77.7 mm to (225.0, 88.5)
- moved H9 70.2 mm to (133.5, 93.0)
- moved H8 37.5 mm to (133.5, 130.5)
- moved H2 31.0 mm to (179.0, 39.5)
- moved H7 26.5 mm to (160.0, 131.0)
- moved R606 3.04 mm to (173.0, 116.5)
- moved R605 2.12 mm to (178.5, 121.5), turned to -90 degrees
- moved C602 1.80 mm to (174.2, 114.9)
- moved C603 1.80 mm to (174.2, 113.4)
- moved R607 1.80 mm to (176.2, 112.9)
- moved R608 1.80 mm to (174.2, 112.4)
- moved Q601 1.00 mm to (174.0, 126.5)
- moved R601 1.00 mm to (182.6, 125.6)
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Routing:
- net Net-(U602-ISET): track 1.88 -> 5.09 mm
- net GND: track 452.0 -> 454.8 mm
- net Net-(Q601-D): track 14.5 -> 11.8 mm
- net POGO_5V: track 36.2 -> 33.6 mm
- net POGO_5V_SENSE: track 46.2 -> 44.4 mm
- net 3V3_PWR: track 348.1 -> 346.7 mm
- net POGO_TX: track 60.0 -> 59.0 mm
- net POGO_RX: track 61.0 -> 60.0 mm
- net POGO_DET: track 71.2 -> 70.5 mm
- net Net-(J601-Pin_3): track 9.21 -> 8.61 mm
