File: hardware/dock-v2/pogo.kicad_sch (KiCad schematic)
At the start: 17 parts, among them J601 Pogo 7-pin, Q601 2N7002, Q602 2N7002, U601 TPD4E1U06DBVR, U602 SY6280AAC

Commit message: Dock v2: J601 becomes a JST-XH 7-pin cable header (pad docks on top)
- pad sits on top of the dock (decided): straight Motorobit 7-pin pogo contacts
  on a small lid board (same design as the pad's pogo board), cabled 1:1 to J601
- J601: B7B-XH-A (LCSC C144398) on the original pin row; 5 V link between
  pins 2/6 moved 0.75 mm lower to clear the larger XH pads; silk trimmed at the edge
- pad MCU decided: ESP32-S3-MINI-1-N8 (README)
- docs: pogo, placement, DESIGN §15/§17, README, generated guides

DRC: 0 violations, 0 unconnected, 0 parity issues.

Co-Authored-By: Claude Opus 5.5 <noreply@anthropic.com>
Parts:
- J601: value Pogo 7-pin -> B7B-XH-A (to lid pogo board); footprint dock:Pogo-7 -> Connector_JST:JST_XH_B7B-XH-A_1x07_P2.50mm_Vertical; LCSC (none) -> C144398; Note HAND-SOLDER: Motorobit 7-pin 90deg magnetic (order: guide §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 -> HAND-SOLDER: JST-XH 7-pin header; 1:1 cable to the pogo boa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
Changed lines of the file:
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@@
 			)
 		)
-		(property "Value" "Pogo 7-pin"
+		(property "Value" "B7B-XH-A (to lid pogo board)"
 			(at 38.1 33.02 0)
 			(show_name no)
@@
 			)
 		)
-		(property "Footprint" "dock:Pogo-7"
+		(property "Footprint" "Connector_JST:JST_XH_B7B-XH-A_1x07_P2.50mm_Vertical"
 			(at 41.91 34.29 0)
 			(hide yes)
@@
 			)
 		)
-		(property "Description" "Generic connector, single row, 01x06, script generated (kicad-library-utils/schlib/autogen/connector/)"
+		(property "Description" ""
 			(at 41.91 34.29 0)
 			(hide yes)
@@
 			)
 		)
-		(property "LCSC" ""
+		(property "LCSC" "C144398"
 			(at 41.91 34.29 0)
 			(hide yes)
@@
 			)
 		)
-		(property "Note" "HAND-SOLDER: Motorobit 7-pin 90deg magnetic (order: guide §8)"
+		(property "Note" "HAND-SOLDER: JST-XH 7-pin header; 1:1 cable to the pogo board in the dock lid (contacts: guide §8)"
 			(at 38.1 30.48 0)
 			(hide yes)

Commit message: Dock v2: J601 uses a project copy of the XH footprint with the silk trimmed at the edge (no library-mismatch warning)
Co-Authored-By: Claude Opus 5.5 <noreply@anthropic.com>
Parts:
- J601: footprint Connector_JST:JST_XH_B7B-XH-A_1x07_P2.50mm_Vertical -> dock:JST_XH_B7B-XH-A_1x07_P2.50mm_Vertical_EdgeTrim
Changed lines of the file:
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@@
 			)
 		)
-		(property "Footprint" "Connector_JST:JST_XH_B7B-XH-A_1x07_P2.50mm_Vertical"
+		(property "Footprint" "dock:JST_XH_B7B-XH-A_1x07_P2.50mm_Vertical_EdgeTrim"
 			(at 41.91 34.29 0)
 			(hide yes)
