File: hardware/pogo/pogo.kicad_sch (KiCad schematic)
At the start: 0 parts

Commit message: Pad: display on 9-pin JST-PH with backlight MOSFET (GP27), pogo cable connector; pogo board schematic; guide updated to final refs
Co-Authored-By: Claude Opus 5.5 <noreply@anthropic.com>
Parts:
- added D1: SMAJ5.0A, Diode_SMD:D_SMA, symbol Device:D_Zener
- added J1: Pogo 6p 90deg (pad half), dock:Pogo-6, symbol Connector_Generic:Conn_01x06
- added J2: Cable to main board, Connector_JST:JST_XH_B4B-XH-A_1x04_P2.50mm_Vertical, symbol Connector_Generic:Conn_01x04
- added U1: TPD4E1U06DBVR, Package_TO_SOT_SMD:SOT-23-6, symbol pad_custom:TPD4E1U06DBV
Connections:
- new net: J1.2 (Pin_2), J2.3 (Pin_3), U1.4 (D2-)
- new net: J1.3 (Pin_3), J2.2 (Pin_2), U1.1 (D1+)
- new net GND: D1.2 (A), J1.1 (Pin_1), J1.4 (Pin_4), J1.6 (Pin_6), J2.1 (Pin_1), U1.2 (GND)
- new net POGO_5V: D1.1 (K), J1.5 (Pin_5), J2.4 (Pin_4)
- no-connect marks 0 -> 2
Other:
- note added: "Pad pogo board: sits vertically in the back wall. Wiring table: hardware/pad/PAD_CONNECTIONS.md section 1a."
- title: Pad pogo board -> (none)

Commit message: 7-pin pogo (2 x +5V, 2 x GND), README and DESIGN for the v2 dock
Pogo: both halves move from the 6-pin to the Motorobit 7-pin 2.54 mm magnetic
set (1 A per contact). Dock side GND | +5V | +5V | DET | RX | TX | GND, pad side
mirrored. New footprint dock:Pogo-7 (scaled from Pogo-6, marked through-hole).
Dock J601 -> Conn_01x07; pogo switch R606 6.8k -> 4.7k (1.45 A, 1.09-1.81 A,
below the 2 A of two contacts), so the pad no longer has to dim its LEDs while
docked. Pad pogo board J1 -> 7 pins, pins 5+6 = POGO_5V, pin 7 = GND (nets
verified before/after). Connection model, guide, pogo/power/placement docs and
PAD_CONNECTIONS updated.

README and DESIGN rewritten for the v2 dock (sections 1-7, 15-22); the pad
sections 8-14 are kept as the v1 plan, to be redesigned. v1 dock stays on master.

Co-Authored-By: Claude Opus 5.5 <noreply@anthropic.com>
Parts:
- J1: footprint dock:Pogo-6 -> dock:Pogo-7; symbol Connector_Generic:Conn_01x06 -> Connector_Generic:Conn_01x07
Connections:
- net GND: now also J1.7 (Pin_7); no longer J1.6 (Pin_6)
- net POGO_5V: now also J1.6 (Pin_6)
Changed lines of the file:
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@@
 	)
 	(junction
-		(at 45.72 55.88)
+		(at 45.72 53.34)
 		(diameter 0)
 		(color 0 0 0 0)
@@
 	(wire
 		(pts
-			(xy 45.72 50.8) (xy 45.72 55.88)
+			(xy 45.72 55.88) (xy 45.72 58.42)
+		)
+		(stroke
+			(width 0)
+			(type default)
+		)
+	)
+	(junction
+		(at 45.72 58.42)
+		(diameter 0)
+		(color 0 0 0 0)
+	)
+	(wire
+		(pts
+			(xy 45.72 50.8) (xy 45.72 53.34)
 		)
 		(stroke
@@
 	)
 	(symbol
-		(lib_id "Connector_Generic:Conn_01x06")
-		(at 40.64 63.5 180)
+		(lib_id "Connector_Generic:Conn_01x07")
+		(at 40.64 60.96 180)
 		(unit 1)
 		(body_style 1)
@@
 		(dnp no)
 		(property "Reference" "J1"
-			(at 40.64 72.39 0)
+			(at 40.64 69.85 0)
 			(show_name no)
 			(do_not_autoplace no)
@@
 		)
 		(property "Value" "Pogo 6p 90deg (pad half)"
-			(at 37.846 63.246 90)
-			(show_name no)
-			(do_not_autoplace no)
-			(effects
-				(font
-					(size 1.27 1.27)
-				)
-			)
-		)
-		(property "Footprint" "dock:Pogo-6"
-			(at 40.64 63.5 0)
+			(at 37.846 60.71 90)
+			(show_name no)
+			(do_not_autoplace no)
+			(effects
+				(font
+					(size 1.27 1.27)
+				)
+			)
+		)
+		(property "Footprint" "dock:Pogo-7"
+			(at 40.64 60.96 0)
 			(hide yes)
 			(show_name no)
@@
 		)
 		(property "Datasheet" ""
-			(at 40.64 63.5 0)
+			(at 40.64 60.96 0)
 			(hide yes)
 			(show_name no)
@@
 		)
 		(property "Description" "Generic connector, single row, 01x06, script generated (kicad-library-utils/schlib/autogen/connector/)"
-			(at 40.64 63.5 0)
+			(at 40.64 60.96 0)
 			(hide yes)
 			(show_name no)
@@
 		)
 		(pin "6"
+		)
+		(pin "7"
 		)
 		(instances
@@
 	(symbol
 		(lib_id "power:GND")
-		(at 45.72 55.88 90)
+		(at 45.72 53.34 90)
 		(unit 1)
 		(body_style 1)
@@
 		(fields_autoplaced yes)
 		(property "Reference" "#PWR02"
-			(at 52.07 55.88 0)
+			(at 52.07 53.34 0)
 			(hide yes)
 			(show_name no)
@@
 		)
 		(property "Value" "GND"
-			(at 49.53 55.8799 90)
+			(at 49.53 53.34 90)
 			(show_name no)
 			(do_not_autoplace no)
@@
 		)
 		(property "Footprint" ""
-			(at 45.72 55.88 0)
+			(at 45.72 53.34 0)
 			(hide yes)
 			(show_name no)
@@
 		)
 		(property "Datasheet" ""
-			(at 45.72 55.88 0)
+			(at 45.72 53.34 0)
 			(hide yes)
 			(show_name no)
@@
 		)
 		(property "Description" "Power symbol creates a global label with name \"GND\" , ground"
-			(at 45.72 55.88 0)
-			(hide yes)
-			(show_name no)
+			(at 45.72 53.34 0)
+			(hide yes)
+			(show_name no)

Commit message: Pogo order GND | +5V | DET | RX | TX | +5V | GND (5 V at both ends)
The dock's J601 now has +5V on pins 2 and 6, like GND on 1 and 7 (user's change
in the schematic). Pad side mirrors to GND | +5V | TX | RX | DET | +5V | GND.
Power pins are mirror-symmetric, so a reversed pad is still powered correctly;
only the UART lines cross (through 1 kOhm, harmless).

- connection model: J601 pins and the U601 ESD channels as wired
- guides regenerated (DOCK_CONNECTIONS, DOCK_WIRING); generators now list parts
  that aren't in the schematic instead of failing
- pad pogo board (hardware/pogo) rewired to the mirrored order with labels;
  nets verified (POGO_5V J1.2/J1.6, DTX J1.3, DRX J1.4, GND J1.1/5/7), ERC clean;
  value "Pogo 7p"
- pogo doc, DESIGN §15, README, PAD_CONNECTIONS §1a updated

Co-Authored-By: Claude Opus 5.5 <noreply@anthropic.com>
Parts:
- J1: value Pogo 6p 90deg (pad half) -> Pogo 7p 90deg (pad half)
Connections:
- net GND: now also J1.5 (Pin_5); no longer J1.4 (Pin_4)
- net POGO_5V: now also J1.2 (Pin_2); no longer J1.5 (Pin_5)
- net POGO_DTX: now reaches J2.3 (Pin_3), U1.4 (D2-)
- net POGO_DTX: now also J1.3 (Pin_3); no longer J1.2 (Pin_2)
- net POGO_DRX: now reaches J2.2 (Pin_2), U1.1 (D1+)
- net POGO_DRX: now also J1.4 (Pin_4); no longer J1.3 (Pin_3)
Changed lines of the file:
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@@
-	)
-	(junction
-		(at 55.88 58.42)
-		(diameter 0)
-		(color 0 0 0 0)
 	)
 	(junction
@@
 	(wire
 		(pts
-			(xy 55.88 58.42) (xy 45.72 58.42)
-		)
-		(stroke
-			(width 0)
-			(type default)
-		)
-	)
-	(wire
-		(pts
 			(xy 64.77 68.58) (xy 64.77 66.04)
 		)
@@
 	(wire
 		(pts
-			(xy 72.39 63.5) (xy 45.72 63.5)
+			(xy 59.69 63.5) (xy 72.39 63.5)
 		)
 		(stroke
@@
 	(wire
 		(pts
-			(xy 64.77 66.04) (xy 45.72 66.04)
+			(xy 59.69 66.04) (xy 64.77 66.04)
 		)
 		(stroke
@@
 			(type default)
 		)
-	)
-	(wire
-		(pts
-			(xy 45.72 55.88) (xy 45.72 58.42)
-		)
-		(stroke
-			(width 0)
-			(type default)
-		)
-	)
-	(junction
-		(at 45.72 58.42)
-		(diameter 0)
-		(color 0 0 0 0)
 	)
 	(wire
@@
 			)
 			(justify right bottom)
+		)
+	)
+		(label "POGO_5V"
+		(at 45.72 66.04 0)
+		(effects
+			(font
+				(size 1.27 1.27)
+			)
+			(justify left bottom)
+		)
+	)
+		(label "POGO_DTX"
+		(at 45.72 63.5 0)
+		(effects
+			(font
+				(size 1.27 1.27)
+			)
+			(justify left bottom)
+		)
+	)
+		(label "POGO_DRX"
+		(at 45.72 60.96 0)
+		(effects
+			(font
+				(size 1.27 1.27)
+			)
+			(justify left bottom)
+		)
+	)
+		(label "POGO_5V"
+		(at 45.72 55.88 0)
+		(effects
+			(font
+				(size 1.27 1.27)
+			)
+			(justify left bottom)
+		)
+	)
+		(label "POGO_DTX"
+		(at 59.69 66.04 0)
+		(effects
+			(font
+				(size 1.27 1.27)
+			)
+			(justify left bottom)
+		)
+	)
+		(label "POGO_DRX"
+		(at 59.69 63.5 0)
+		(effects
+			(font
+				(size 1.27 1.27)
+			)
+			(justify left bottom)
 		)
 	)
@@
 	(symbol
 		(lib_id "power:GND")
-		(at 45.72 60.96 90)
+		(at 45.72 58.42 90)
 		(unit 1)
 		(body_style 1)
@@
 		(fields_autoplaced yes)
 		(property "Reference" "#PWR05"
-			(at 52.07 60.96 0)
+			(at 52.07 58.42 0)
 			(hide yes)
 			(show_name no)
@@
 		)
 		(property "Value" "GND"
-			(at 49.53 60.9599 90)
+			(at 49.53 58.42 90)
 			(show_name no)
 			(do_not_autoplace no)
@@
 		)
 		(property "Footprint" ""
-			(at 45.72 60.96 0)
+			(at 45.72 58.42 0)
 			(hide yes)
 			(show_name no)
@@
 		)
 		(property "Datasheet" ""
-			(at 45.72 60.96 0)
+			(at 45.72 58.42 0)
 			(hide yes)
 			(show_name no)
@@
 		)
 		(property "Description" "Power symbol creates a global label with name \"GND\" , ground"
-			(at 45.72 60.96 0)
+			(at 45.72 58.42 0)
 			(hide yes)
 			(show_name no)
@@
 			)
 		)
-		(property "Value" "Pogo 6p 90deg (pad half)"
+		(property "Value" "Pogo 7p 90deg (pad half)"
 			(at 37.846 60.71 90)
 			(show_name no)
