File: hardware/pad-v2/rgb.kicad_sch (KiCad schematic)
At the start: 83 parts, among them U401 TPS61023DRLR, U402 SN74AHCT1G125DBVR

Commit message: Pad v2: GPIO map for routing, PAD_WIRING.md (component-by-component), connection model + checker; battery 2-pin + NTC header, USB-C to the front edge, LED chain starts at key 9
Co-Authored-By: Claude Opus 5.5 <noreply@anthropic.com>
Parts:
- removed D401, D402, D403, D404, D405, D406, D407, D408, D409, D410, D411, D412: XL-2020RGBC-WS2812B, pad_v2:LED_XL-2020RGBC_2.0x2.0mm, symbol LED:WS2812B-2020
- removed D413, D414, D415, D416, D429, D430, D431, D432, D433, D434, D435, D436: SK6812MINI-E, LED_SMD:LED_SK6812MINI-E_3.2x2.8mm_P1.5mm_ReverseMount, symbol LED:SK6812MINI-E
- added D401, D402, D403, D404, D405, D406, D407, D408, D409, D410, D411, D412: SK6812MINI-E, LED_SMD:LED_SK6812MINI-E_3.2x2.8mm_P1.5mm_ReverseMount, symbol LED:SK6812MINI-E
- added D413, D414, D415, D416, D429, D430, D431, D432, D433, D434, D435, D436: XL-2020RGBC-WS2812B, pad_v2:LED_XL-2020RGBC_2.0x2.0mm, symbol LED:WS2812B-2020
- D417: Note chain index 16: ring 2, 7 o'clock -> chain index 16: ring 2, 3 o'clock
- D418: Note chain index 17: ring 2, 8 o'clock -> chain index 17: ring 2, 2 o'clock
- D419: Note chain index 18: ring 2, 9 o'clock -> chain index 18: ring 2, 1 o'clock
- D420: Note chain index 19: ring 2, 10 o'clock -> chain index 19: ring 2, 12 o'clock
- D422: Note chain index 21: ring 2, 12 o'clock -> chain index 21: ring 2, 10 o'clock
- D423: Note chain index 22: ring 2, 1 o'clock -> chain index 22: ring 2, 9 o'clock
- D424: Note chain index 23: ring 2, 2 o'clock -> chain index 23: ring 2, 8 o'clock
- D425: Note chain index 24: ring 2, 3 o'clock -> chain index 24: ring 1, 4 o'clock
- D426: Note chain index 25: ring 2, 4 o'clock -> chain index 25: ring 1, 3 o'clock
- D427: Note chain index 26: ring 2, 5 o'clock -> chain index 26: ring 1, 2 o'clock
- D428: Note chain index 27: ring 2, 6 o'clock -> chain index 27: ring 1, 1 o'clock
- R404: Note series, U402 output to D401 DIN -> series, U402 output to D401 DIN (key 9 LED)
- U401: Note VSYS -> 5V_RGB; EN from a GPIO (true disconnect when low) -> VSYS -> 5V_RGB; EN = RGB_EN (IO26), true disconnect when low
- U402: Note powered from 5V_RGB; OE to GND -> input RGB_DATA (IO46); powered from 5V_RGB; OE (pin 1) to G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
Other:
- note added: "Key LEDs: keys 1, 2, 3, 4"
- note added: "Key LEDs: keys 8, 7, 6, 5"
- note added: "Key LEDs: keys 9, 10, 11, 12 (chain starts here)"
- note added: "Ring 1 (ENC1), counter-clockwise from 4 o'clock"
- note added: "Ring 2 (ENC2), counter-clockwise from 7 o'clock"
- note removed: "Key LEDs, keys 1-4"
- note removed: "Key LEDs, keys 8, 7, 6, 5"
- note removed: "Key LEDs, keys 9-12"
- note removed: "Ring 1 (ENC1), clockwise from 6 o'clock"
- note removed: "Ring 2 (ENC2), clockwise from 7 o'clock"
